File: bi-directional-amp-board/Bidirectional_Amp.brd (EAGLE design)
At the start: 78.5 x 52 mm, 135 parts, among them J1 73415-2061, J10 73415-2061, J11 73415-2061, J12 73415-2061, J2 73415-2061, J4 73415-2061, J5 73415-2061, J6 73415-2061, J7 73415-2061, J8 73415-2061, U1 LTC5536, U10 NC7S32M5X, U11 SN74LV1T34DBVR, U12 LTC3428EDDPBF, U2 LTC6994-1, U3 LTC6994-1, U4 QPC1022, U5 NC7S04M5, U6 TQP9111, U7 TQP3M9035, U8 QPC1022

Commit message: mawr
Parts:
- removed C45: 22pF, rcl:C0402
- added C38: 22pF, oresat-rcl:.0402-B-NOSILK
- C1, C10, C11, C12, C13, C14, C2, C27, C3, C30, C31, C32, C33, C36, C39, C4, C40, C41, C42, C5, C6, C7, C8, C9: device rcl:C0402 -> oresat-rcl:.0402-B-NOSILK
- C18: value 100nF -> 100pF
- moved CF1 13.4 mm to (62.0, 12.0), turned to 90 degrees
- moved J8 13.4 mm to (62.0, 17.0), turned to 90 degrees
- moved J12 13.3 mm to (62.0, 23.0), turned to 90 degrees
- moved J7 8.99 mm to (66.4, 29.0)
- moved J11 7.46 mm to (68.0, 35.0)
- moved R33 4.12 mm to (66.0, 17.0), turned to 180 degrees
- moved R34 4.12 mm to (66.0, 12.0), turned to 180 degrees
- moved R38 4.00 mm to (66.0, 23.0), turned to 180 degrees
- moved C42 3.92 mm to (65.0, 35.0)
- moved FL3 2.48 mm to (69.5, 41.3)
- moved J4 2.48 mm to (75.6, 41.3)
- moved J5 2.48 mm to (62.0, 41.0)
- moved L11 2.48 mm to (72.0, 41.8)
- moved L12 2.48 mm to (67.5, 40.4)
- moved R35 2.48 mm to (65.5, 41.0)
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- renumbered C43 to C34, C44 to C37, C46 to C25, C47 to C35, D3 to D1, D4 to D2, J13 to J3, L13 to L9, L14 to L10, R40 to R28, R41 to R29, R42 to R30, R43 to R31, U12 to U9
Connections:
- net GND: now also C38.2; no longer C45.2
- net VC1: now also C38.1; no longer C45.1
Routing:
- net N$47: track 13.5 -> 4.38 mm
- net GND: track 93.6 -> 88.3 mm, vias 531 -> 532
- net N$53: track 6.16 -> 2.50 mm
- net N$54: track 6.04 -> 2.50 mm
- net N$19: track 2.53 -> 0.58 mm
- net N$20: track 1.97 -> 0.46 mm
- net N$55: track 4.46 -> 3.15 mm
- net N$49: track 4.46 -> 3.15 mm
- net N$48: track 4.46 -> 3.15 mm
- net +5V: track 40.3 -> 39.3 mm
- added copper zone on layer 1, net N$19
- added copper zone on layer 1, net N$20

Commit message: more adds
Routing:
- net N$17: track 6.56 -> 0.00 mm
- net N$13: track 9.57 -> 3.37 mm
- net GND: track 88.3 -> 83.8 mm, vias 532 -> 553
- net +5V: track 39.3 -> 38.5 mm, vias 21 -> 23
- net N$39: track 0.00 -> 0.18 mm, vias 0 -> 1
- net VOUT1: vias 0 -> 6
- net VIN1: vias 2 -> 8
- added copper zone on layer 1, net +5V

Commit message: a few updates
Parts:
- removed U$1: (no value), Oliver_Custom:PSAS_LOGO_10X10_NEW
- moved L10 0.46 mm to (44.3, 10.3), turned to 270 degrees
Routing:
- net VIN1: track 4.75 -> 1.08 mm, vias 8 -> 7
- net GND: track 83.8 -> 86.4 mm, vias 553 -> 565
- removed copper zone on layer 1, net SWB1
Other:
- board text added: "AUTO"
- board text added: "NUMBER THESE"
- board text added: "RX"
- board text added: "TX"
- board text added: "WINDOW TCREAM"

Commit message: added more revisions
Parts:
- moved J12 6.50 mm to (68.5, 23.0)
- moved J8 6.50 mm to (68.5, 17.0)
- moved R33 6.50 mm to (72.5, 17.0)
- moved R38 6.50 mm to (72.5, 23.0)
- moved J6 4.34 mm to (66.3, 29.0)
- moved J7 4.34 mm to (70.7, 29.0)
- moved C42 3.53 mm to (68.5, 35.0)
- moved J10 3.53 mm to (65.5, 35.0)
- moved J11 3.53 mm to (71.5, 35.0)
- moved CF1 1.48 mm to (63.1, 11.0)
- moved R34 1.48 mm to (67.1, 11.0)
- moved R2 1.06 mm to (19.1, 45.0), turned to 180 degrees
Routing:
- net +5V: track 38.5 -> 25.0 mm
- net N$18: track 35.4 -> 22.0 mm, vias 2 -> 1
- net N$34: track 7.07 -> 2.25 mm
- net VIN1: track 1.08 -> 5.35 mm, vias 7 -> 8
- net N$17: track 0.00 -> 2.03 mm
- net N$10: track 44.5 -> 45.6 mm
- net N$13: track 3.37 -> 4.37 mm
- net N$32: track 10.5 -> 9.71 mm
- net GND: track 86.4 -> 86.2 mm, vias 565 -> 890
- net N$39: track 0.18 -> 0.00 mm, vias 1 -> 0
- added copper zone on layer 1, net SWB1
Other:
- board text added: "1"
- board text added: "2"
- board text added: "2.4GHz WiFi BPF"
- board text added: "3"
- board text added: "4"
- board text added: "5"
- board text added: "6"
- board text added: "7"
- board text added: "8"
- board text added: "COUPLING CAP"
- board text added: "HF RESISTOR"
- board text added: "ORESAT DxWiFi PA/LNA BOARD OLIVER JONES OLIVER REW 2018-09-05"
- board text added: "STD RESISTOR"
- board text added: "STUB"
- board text added: "TESTS"
- board text added: "THROUGH"
- board text removed: "NUMBER THESE"
- board text removed: "WINDOW TCREAM"

Commit message: more refinements
Parts:
- moved S1 0.75 mm to (16.0, 14.8)
- moved J6 0.50 mm to (65.8, 29.0)
- moved J7 0.50 mm to (71.2, 29.0)
- moved R24 0.31 mm to (39.6, 37.5)
- moved R25 0.31 mm to (40.6, 37.5)
- moved R26 0.31 mm to (42.6, 37.5), turned to 90 degrees
- moved R27 0.31 mm to (41.6, 37.5), turned to 270 degrees
- moved C32 0.19 mm to (43.6, 37.5), turned to 270 degrees
- moved R13 0.19 mm to (22.4, 37.5)
- moved R14 0.19 mm to (21.4, 37.5)
- moved R15 0.19 mm to (19.4, 37.5), turned to 270 degrees
- moved R16 0.19 mm to (20.4, 37.5), turned to 90 degrees
- moved C11 0.16 mm to (18.4, 37.5), turned to 90 degrees
- moved C12 0.12 mm to (17.4, 37.5)
- moved C33 0.12 mm to (44.6, 37.5)
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Routing:
- net N$18: track 22.0 -> 35.9 mm, vias 1 -> 2
- net N$17: track 2.03 -> 7.59 mm
- net N$13: track 4.37 -> 9.77 mm
- net N$34: track 2.25 -> 7.65 mm
- net +5V: track 25.0 -> 21.7 mm
- net N$47: track 4.38 -> 5.38 mm
- net N$52: track 5.98 -> 5.23 mm
- net N$10: track 45.6 -> 46.3 mm
- net FORCE_BRDCST_+3.3V: track 32.3 -> 31.6 mm
- net GND: track 86.2 -> 86.3 mm, vias 890 -> 897
Other:
- board text added: "FORCE TX"
- board text added: "ORESAT DxWiFi PA/LNA BOARD REV.1 OLIVER JONES OLIVER REW 2018-09-05"
- board text removed: "ORESAT DxWiFi PA/LNA BOARD OLIVER JONES OLIVER REW 2018-09-05"

Commit message: argggggg
Routing:
- net GND: vias 897 -> 895
Changed lines of the file:
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@@
 <via x="42.125" y="34.21875" extent="1-16" drill="0.127" diameter="0.001"/>
 <via x="48" y="37.5" extent="1-16" drill="0.127" diameter="0.001"/>
-<via x="48.1875" y="37.8125" extent="1-16" drill="0.127" diameter="0.001"/>
-<via x="48.1875" y="37.1875" extent="1-16" drill="0.127" diameter="0.001"/>
 <via x="48.5625" y="36.9375" extent="1-16" drill="0.127" diameter="0.001"/>
 <via x="48.5625" y="38.0625" extent="1-16" drill="0.127" diameter="0.001"/>

Commit message: changes from design review
Parts:
- moved LED1 21.1 mm to (28.5, 14.2)
- moved LED2 21.1 mm to (32.0, 14.2)
- moved R32 21.1 mm to (28.5, 17.0)
- moved R36 21.1 mm to (32.0, 17.0)
Routing:
- net N$10: track 46.3 -> 30.2 mm, vias 0 -> 2
- net PA_ON_LNA_OFF: track 34.1 -> 20.2 mm
- net N$18: track 35.9 -> 27.5 mm
- net TX_RX_CTL: track 27.0 -> 21.3 mm
- net +5V: track 21.7 -> 19.0 mm, vias 23 -> 24
- net VC1: track 7.39 -> 9.13 mm
- net N$3: track 2.45 -> 2.97 mm
- net SHDN1: track 17.3 -> 16.8 mm
- net FORCE_BRDCST_+5V: track 7.87 -> 8.05 mm, vias 0 -> 2
- net GND: track 86.3 -> 86.2 mm, vias 895 -> 566
Other:
- outline, holes or cut-outs redrawn
- board text added: "PWR"

Commit message: could be the final rev!
Parts:
- moved LED1 3.50 mm to (26.5, 17.1), turned to 180 degrees
- moved LED2 2.97 mm to (31.2, 17.1), turned to 180 degrees
- moved S1 2.75 mm to (13.2, 14.8)
- moved R32 2.58 mm to (26.5, 18.6), turned to 0 degrees
- moved R36 1.79 mm to (31.2, 18.6), turned to 0 degrees
- moved CF1 0.88 mm to (62.2, 11.0)
- moved R34 0.88 mm to (66.2, 11.0)
Routing:
- net N$10: track 30.2 -> 28.3 mm
- net FORCE_BRDCST_+3.3V: track 31.6 -> 33.2 mm
- net GND: track 86.2 -> 87.7 mm, vias 566 -> 588
- net N$52: track 5.23 -> 6.27 mm
- net N$18: track 27.5 -> 28.5 mm
- net N$19: track 0.58 -> 0.00 mm
Other:
- board text added: "!DISABLE"
- board text added: "5V EXT"
- board text added: "5V OUT"
- board text added: "5V PWR"
- board text added: "ANT"
- board text added: "GND"
- board text added: "HOST"
- board text added: "OLIVER JONES OLIVER REW 2018-09-07"
- board text added: "ORESAT DxWiFi PA/LNA BOARD REV.1"
- board text added: "POWER HEADER"
- board text added: "VBAT"
- board text removed: "ORESAT DxWiFi PA/LNA BOARD REV.1 OLIVER JONES OLIVER REW 2018-09-05"
