File: pa-test-board/Bidirectional_Amp_test.sch (EAGLE design)
At the start: 34 parts, among them J1 142-0701-851, J2 142-0701-851, J3 142-0701-851, J4 142-0701-851, SW1 TL36PO, U10 TQP9111

Commit message: Attribues added to parts and BOMs created via ULP
Parts:
- C15, C16, C17: DESCRIPTION (none) -> CAP CER 0.1UF 16V X7R 0402
- C18: DESCRIPTION (none) -> CAP CER 0.1UF 16V X7R 0402; MFR Murata -> TDK; MPN GCM1555C1H101JA16D -> CGA2B1X7R1C104K050BC
- C19: DESCRIPTION (none) -> CAP CER 1000PF 50V NP0 0402
- C20: DESCRIPTION (none) -> CAP CER 100PF 50V C0G/NP0 0603
- C21: DESCRIPTION (none) -> CAP CER 3PF 50V NP0 0402; MFR Taiyo Yuden -> AVX; MPN UVK105CG030JW-F -> 04025U3R0BAT2A
- C22: DESCRIPTION (none) -> Capacitor Thin Film 50V 2.5pF .03pFTol 0402; MFR Taiyo Yuden -> AVX; MPN UVK105CG2R2JW-F -> 04025J2R5QBSTR
- C23: DESCRIPTION (none) -> CAP CER 1.6PF 50V NP0 0402; MFR Murata -> AVX; MPN GJM1555C1H1R6BB01D -> 04025U1R6BAT2A
- C34: DESCRIPTION (none) -> CAP CER 4.7UF 16V X7R 1206; SIZE 1206 -> (none); VOLTAGE 16V -> (none)
- C35: DESCRIPTION (none) -> CAP CER 22UF 16V X7R 1210
- J1, J2, J3, J4: DESCRIPTION (none) -> CONN SMA JACK STR 50OHM EDGE MNT; MFR (none) -> Cinch Connectivity Solutions Johnson; MPN (none) -> 142-0701-851
- JP6: DESCRIPTION (none) -> CONN HEADER VERT 4POS 2.54MM; MFR (none) -> Molex; MPN (none) -> 0022232041
- L2: DESCRIPTION (none) -> Fixed Inductors 080xSQ AirCore RF 10.2 nH 2 % 2.7 A; MFR CoilCraft -> Coilcraft; MPN 0807SQ-10n -> 0807SQ-10NGLB
- L3: value 1.2nH -> 1.0nH; DESCRIPTION (none) -> FIXED IND 1NH 500MA 100 MOHM SMD; MFR (none) -> TDK Corporation; MPN (none) -> MLK1005S1N0ST000
- L4: DESCRIPTION (none) -> 1.2nH RF Inductor, ceramic core, 5% tol, SMT, RoHS, halogen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; MFR (none) -> Coilcraft; MPN (none) -> 0402CT-1N2XJRW
- L5: DESCRIPTION (none) -> Fixed Inductors 0805CS 6.8 nH 5 % 0.6 A; MFR (none) -> Coilcraft; MPN (none) -> 0805CS-060XJLC
- R1: DESCRIPTION (none) -> RES SMD 0 OHM JUMPER 1/10W 0402; MFR (none) -> Panasonic Electronic Components; MPN (none) -> ERJ-2GE0R00X
- R17: DESCRIPTION (none) -> RES SMD 0 OHM JUMPER 1/8W 0805
- R19: DESCRIPTION (none) -> RES SMD 110 OHM 1% 1/10W 0402
- R20: DESCRIPTION (none) -> RES SMD 220 OHM 1% 1/10W 0603
- R32, R36: DESCRIPTION (none) -> RES SMD 1K OHM 5% 1/10W 0402
- SW1: DESCRIPTION (none) -> SWITCH TOGGLE SPDT 0.4VA 20V
