File: pa-test-board_V2/pa-test-board_V2.brd (EAGLE design)
At the start: 30 x 44 mm, 34 parts, among them J1 142-0701-851, J2 142-0701-851, J3 142-0701-851, J4 142-0701-851, SW1 TL36PO, U10 TQP9111

Commit message: Updated to tuned values, fixed BOM formatting.
Parts:
- C22: value 1.2pF -> 1.1pF
Changed lines of the file:
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@@
 <attribute name="VALUE" x="17.095" y="32.685" size="1.27" layer="27" rot="R270"/>
 </element>
-<element name="C22" library="oresat-rcl" package=".0402-C-NOSILK" value="1.2pF" x="9.6" y="32.5" smashed="yes">
-<attribute name="DESCRIPTION" value="Capacitor Thin Film 50V 1.2pF .02pFTol  0402" x="9.6" y="32.5" size="1.778" layer="27" display="off"/>
+<element name="C22" library="oresat-rcl" package=".0402-C-NOSILK" value="1.1pF" x="9.6" y="32.5" smashed="yes">
+<attribute name="DESCRIPTION" value="50V 1.1pF .02pFTol ThinFilm 0402" x="9.6" y="32.5" size="1.778" layer="27" display="off"/>
 <attribute name="MFR" value="AVX" x="9.6" y="32.5" size="1.778" layer="27" display="off"/>
-<attribute name="MPN" value="04025J1R2PBSTR" x="9.6" y="32.5" size="1.778" layer="27" display="off"/>
+<attribute name="MPN" value="04025J1R1PBSTR\500" x="9.6" y="32.5" size="1.778" layer="27" display="off"/>
 <attribute name="NAME" x="8.84625" y="29.6960625" size="0.635" layer="25" font="vector" ratio="20"/>
 <attribute name="VALUE" x="8.965" y="30.595" size="1.27" layer="27"/>
@@
 <attribute name="MFR" value="Coilcraft" x="8.2" y="32.05" size="1.778" layer="27" rot="R90" display="off"/>
 <attribute name="MPN" value="0402DC-1N7XJRU" x="8.2" y="32.05" size="1.778" layer="27" rot="R90" display="off"/>
+<attribute name="NAME" x="8.4" y="29.55" size="0.635" layer="25" font="vector" ratio="20" rot="R90"/>
 <attribute name="NAME" x="8.2" y="32.05" size="0.2" layer="33" ratio="15" rot="R90" align="center"/>
-<attribute name="NAME" x="8.4" y="29.55" size="0.635" layer="25" font="vector" ratio="20" rot="R90"/>
 <attribute name="VALUE" x="9.6" y="31.35" size="0.8" layer="27" font="vector" ratio="15" rot="R90"/>
 </element>
@@
 <attribute name="MFR" value="Coilcraft" x="11.8" y="36.4" size="1.778" layer="27" rot="R180" display="off"/>
 <attribute name="MPN" value="0805CS-060XJLC" x="11.8" y="36.4" size="1.778" layer="27" rot="R180" display="off"/>
+<attribute name="NAME" x="10.65" y="37.25" size="0.635" layer="25" font="vector" ratio="20"/>
 <attribute name="NAME" x="11.8" y="36.4" size="0.4" layer="33" ratio="15" rot="R180" align="center"/>
-<attribute name="NAME" x="10.65" y="37.25" size="0.635" layer="25" font="vector" ratio="20"/>
 <attribute name="VALUE" x="13.05" y="38.05" size="0.8" layer="27" font="vector" ratio="15" rot="R180"/>
 </element>
@@
 <attribute name="MFR" value="TDK Corporation" x="20.4" y="32.5" size="1.778" layer="27" display="off"/>
 <attribute name="MPN" value="MLK1005S1N0ST000" x="20.4" y="32.5" size="1.778" layer="27" display="off"/>
+<attribute name="NAME" x="20.4" y="32.5" size="0.2" layer="33" ratio="15" align="center"/>
 <attribute name="NAME" x="20.1" y="29.75" size="0.635" layer="25" font="vector" ratio="20"/>
-<attribute name="NAME" x="20.4" y="32.5" size="0.2" layer="33" ratio="15" align="center"/>
 <attribute name="VALUE" x="19.7" y="31.25" size="0.8" layer="27" font="vector" ratio="15"/>
 </element>
@@
 <attribute name="MFR" value="Vishay / Dale" x="11.4" y="32.5" size="1.778" layer="27" display="off"/>
 <attribute name="MPN" value="CRCW04023R30FKED" x="11.4" y="32.5" size="1.778" layer="27" display="off"/>
+<attribute name="NAME" x="11.1" y="29.75" size="0.635" layer="25" font="vector" ratio="20"/>
 <attribute name="NAME" x="11.4" y="32.5" size="0.2" layer="33" ratio="15" align="center"/>
-<attribute name="NAME" x="11.1" y="29.75" size="0.635" layer="25" font="vector" ratio="20"/>
 <attribute name="VALUE" x="10.7" y="31.25" size="0.8" layer="27" font="vector" ratio="15"/>
 </element>
