File: wf-np9202-carrier/wf-np9202-carrier.sch (EAGLE design)
At the start: 17 parts, among them J1 UJ2-MIBH2-4-SMT-TR, J3 SM06B-SRSS-TB(LF)(SN)

Commit message: Minor updates, changed BOM filename.
Other:
- note added: "ID should float (device, not host)"
Changed lines of the file:
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@@
 <setting verticaltext="up"/>
 </settings>
-<grid distance="0.05" unitdist="inch" unit="inch" style="lines" multiple="1" display="no" altdistance="0.01" altunitdist="inch" altunit="inch"/>
+<grid distance="0.05" unitdist="inch" unit="inch" style="lines" multiple="2" display="no" altdistance="0.01" altunitdist="inch" altunit="inch"/>
 <layers>
 <layer number="1" name="Top" color="4" fill="1" visible="no" active="no"/>
@@
 2.4 GHz PCB Antenna
 (with adhesive)</text>
+<text x="69.85" y="124.46" size="1.778" layer="97">ID should float (device, not host)</text>
 </plain>
 <instances>
