File: oresat-live-card/KiCAD/OSD3358_USB,_JTAG,_XTAL,_etc_%3a_SIP_B.kicad_sch (KiCad schematic)
At the start: 97 parts, among them J10 SM06B-SRSS-TB(LF)(SN), J8 FTSH-105-XX-X-DV-K, U1 RCLAMP0504FB, U20 TPS2041BQDBVRQ1, U7 OSD3358-512M-BSM, U9 TPS2041BQDBVRQ1, Y1 24MHz, Y2 ABS07-32.768KHZ-T, Y3 6MHz

Commit message: BOM and minor cosmetic schematic updates
Parts:
- removed C61, C62, C? (x2): 50pF, oresat-live-card:.0603-A, symbol oresat-live-card-eagle-import:C-EU0603-A
- removed R93, R95, R? (x2): 22, oresat-live-card:.0603-A, symbol oresat-live-card-eagle-import:R-US_0603-A
- removed R94, R96, R? (x2): 15k, oresat-live-card:.0603-A, symbol oresat-live-card-eagle-import:R-US_0603-A
- removed R? (x2): 10k, oresat-live-card:.0603-A, symbol oresat-live-card-eagle-import:R-US_0603-A
- removed TP169, TP175, TP176, TP181, TP38, TP39: TEST-POINT3X4, oresat-live-card:2MM-TEST-POINT, symbol oresat-live-card-eagle-import:TEST-POINT
- added R90, R91: 10k, Resistor_SMD:R_0603_1608Metric, symbol oresat-live-card-eagle-import:R-US_0603-A
- C1, C28, C4, C42, C7: value 0.1uF -> 100n; footprint oresat-live-card:.0603-A -> Resistor_SMD:R_0603_1608Metric; symbol oresat-live-card-eagle-import:C-EU0603-A -> Device:C_Small; Distributor (none) -> DigiKey; MPN (none) -> CL10B104KB8WPNC
- C19, C22, C29, C30: footprint oresat-live-card:.0603-A -> Resistor_SMD:R_0603_1608Metric; symbol oresat-live-card-eagle-import:C-EU0603-A -> Device:C_Small; Distributor (none) -> DigiKey; MPN (none) -> 06035C120J4T2A
- C24, C25: value 1nF -> 1n; symbol oresat-live-card-eagle-import:C-EU0805-B -> Device:C_Small; Distributor (none) -> DigiKey; MPN (none) -> C0805F102K1RACAUTO
- C26: value 0.1uF -> 100n; symbol oresat-live-card-eagle-import:C-EU0805-B -> Device:C_Small; Distributor (none) -> DigiKey; MPN (none) -> CL21B104KBF5PNE
- C27, C53: value 10uF -> 10u; footprint oresat-live-card:.0603-A -> oresat-live-card:.0805-B; symbol oresat-live-card-eagle-import:C-EU0603-A -> Device:C_Small; Distributor (none) -> DigiKey; MPN (none) -> CGA4J1X7R0J106M125AC
- C54, C55, C56, C57, C58, C59, C60, C65, C66, C67, C68, C70, C71, C72: renamed from C?; footprint Resistor_SMD:R_0603_1608Metric -> oresat-live-card:.0402-B-NOSILK; Distributor (none) -> DigiKey; MPN (none) -> CGJ2B3X7R1E104K050BB
- C63, C64: value 20pF -> 10p; footprint oresat-live-card:.0603-A -> Resistor_SMD:R_0603_1608Metric; symbol oresat-live-card-eagle-import:C-EU0603-A -> Device:C_Small; Distributor (none) -> Mouser; MPN (none) -> C0603C100F1GACTU
- C69: renamed from C?; footprint Resistor_SMD:R_0603_1608Metric -> oresat-live-card:.0805-B; Distributor (none) -> DigiKey; MPN (none) -> CGA4J1X7R0J106M125AC
- C73: renamed from C?; Distributor (none) -> DigiKey; MPN (none) -> CGA3E1X7R1E105M080AE
- FB1, FB2, FB3: Distributor (none) -> DigiKey; MPN (none) -> BLM18KG300JH1D
- FB4, FB5: renamed from FB?; Distributor (none) -> DigiKey; MPN (none) -> MMZ1608Y221BTD25
- J10: Distributor (none) -> DigiKey; MPN (none) -> SM06B-SRSS-TB(LF)(SN)
- R13: footprint oresat-live-card:.0603-A -> Resistor_SMD:R_0603_1608Metric; Distributor (none) -> DigiKey; MPN (none) -> ERJ-3EKF1004V
- R19, R20, R22, R6, R7: footprint oresat-live-card:.0603-A -> Resistor_SMD:R_0603_1608Metric; Distributor (none) -> DigiKey; MPN (none) -> ERJ-3EKF1002V
- R27: footprint oresat-live-card:.0603-A -> Resistor_SMD:R_0603_1608Metric
- R76, R77, R79, R89: renamed from R?; footprint oresat-live-card:.0603-A -> Resistor_SMD:R_0603_1608Metric; Distributor (none) -> DigiKey; MPN (none) -> ERJ-3EKF1002V
- R78: renamed from R?; footprint oresat-live-card:.0603-A -> Resistor_SMD:R_0603_1608Metric; Distributor (none) -> DigiKey; MPN (none) -> RMCF0603FT9K53
- R83: renamed from R?; footprint oresat-live-card:.0603-A -> Resistor_SMD:R_0603_1608Metric; Distributor (none) -> DigiKey; MPN (none) -> ERJ-3EKF9092V
- TP12, TP138, TP139, TP141, TP144, TP171, TP31: footprint oresat-live-card:2MM-TEST-POINT -> oresat-live-card:PAD.03X.04
- TP13, TP16, TP17, TP18: renamed from TP?; footprint oresat-live-card:2MM-TEST-POINT -> oresat-live-card:PAD.03X.04
- U1: Distributor (none) -> DigiKey; MPN (none) -> RCLAMP0504FBTCT
- U2: renamed from U?; Distributor (none) -> DigiKey; MPN (none) -> TUSB4020BI
- U20, U9: Distributor (none) -> DigiKey; MPN (none) -> TPS2041BQDBVRQ1
- U7: Distributor (none) -> DigiKey; MPN (none) -> OSD3358-512M-BSM
- Y1: Distributor (none) -> DigiKey; MPN (none) -> ECS-240-20-30B-TR
- Y2: Distributor (none) -> DigiKey; MPN (none) -> ABS07-32.768KHZ-T
- Y3: value 6MHz -> 24MHz; Distributor (none) -> DigiKey; MPN (none) -> ECS-240-20-30B-TR
Connections:
- net 1.8V-A is gone; now on net PWR: C24.1, C25.1, C26.1, TP171.1, TP8.1, U7.A7 (SYS_ADC_1P8V), U7.B7 (VREFP), U7.N13 (PMIC_MUX_IN)
- net 5V is gone; now on net PWR: C1.1, C28.1, U20.5 (IN), U9.5 (IN)
- net 3.3V: now also R90.2, R91.2; no longer FB5.2, J8.1 (VTREF), R20.2, R22.2, R6.2, R7.2, R77.1, R79.2
- net USB_CAM_N: now also U2.15 (USB_DM_DN2)
- net USB_CAM_P: now also U2.14 (USB_DP_DN2)
- net USB_WIFI_N: now also U2.42 (USB_DM_DN1)
- net USB_WIFI_P: now also U2.41 (USB_DP_DN1)
- net at U2.6 (PWRCTL2/BATEN2), U9.4 (~{EN}): now also R7.1
- net at U2.5 (OVERCUR1z), U20.3 (~{OC}): now also R91.1; no longer R7.1
- net at U2.4 (PWRCTL1/BATEN1), U20.4 (~{EN}): now also R90.1
- net +1V1 renamed PWR
- net PWR: now also FB5.2, J8.1 (VTREF), R20.2, R22.2, R6.2, R7.2, R77.1, R79.2
Other:
- note added: "TODO: Series capacitance"
- note added: "TODO: check ferrite bead location with datasheet"
- note added: "TODO: double check that 3.3V pullups are fine"
- note added: "TODO:Double check that this pin was fixed so nick doesnt do the crazy thing again"
- note removed: "TODO: Replace with 24MHz Crystal"
- note removed: "TODO: verify this is okay"
- note removed: "VSS_OSC"
- note removed: "XTALIN"
- note removed: "XTALOUT"

Commit message: updated schematic with new 5.5V reg
Parts:
- removed J8: FTSH-105-XX-X-DV-K, oresat-live-card:CON10_2X5_DUK_FTSH, symbol oresat-live-card-eagle-import:FTSH-105-XX-X-DV-K
- removed JP1: JUMPER-SMT_2_NO_SILK, oresat-live-card:SMT-JUMPER_2_NO_SILK, symbol oresat-live-card-eagle-import:JUMPER-SMT_2_NO_SILK
- removed R19, R20, R22: 10k, Resistor_SMD:R_0603_1608Metric, symbol oresat-live-card-eagle-import:R-US_0603-A
- removed TP138, TP139, TP141, TP31: TEST-POINT3X4, oresat-live-card:PAD.03X.04, symbol oresat-live-card-eagle-import:TEST-POINT
- added C75, C76: 10u, oresat-live-card:.0805-B, symbol Device:C_Small
- C54, C55, C56, C57, C58, C59, C60, C65, C66, C67, C68, C70, C71, C72: footprint oresat-live-card:.0402-B-NOSILK -> Resistor_SMD:R_0603_1608Metric; MPN CGJ2B3X7R1E104K050BB -> CL10B104KB8WPNC
- C63, C64: value 10p -> 12pF, 50V; Distributor Mouser -> DigiKey; MPN C0603C100F1GACTU -> 06035C120J4T2A
- JP100: footprint oresat-live-card:SMT-JUMPER_2_NC_TRACE_SILK -> Jumper:SolderJumper-2_P1.3mm_Bridged_RoundedPad1.0x1.5mm
- TP1, TP10, TP15, TP8: footprint oresat-live-card:2MM-TEST-POINT -> oresat-live-card:PAD.03X.04
- Y3: footprint oresat-live-card:ECS_ECS-060-18-20BM-JEN-TR -> oresat-live-card:5X3.2-4SMD
Connections:
- net 3.3V: now also FB5.2, R6.2, R7.2, R77.1, R79.2
- net GND: now also C75.2, C76.2
- net USB_CAM_N: now also U2.42 (USB_DM_DN1); no longer U2.15 (USB_DM_DN2)
- net USB_CAM_P: now also U2.41 (USB_DP_DN1); no longer U2.14 (USB_DP_DN2)
- net USB_WIFI_N: now also U2.15 (USB_DM_DN2); no longer U2.42 (USB_DM_DN1)
- net USB_WIFI_P: now also U2.14 (USB_DP_DN2); no longer U2.41 (USB_DP_DN1)
- net at C27.1, C7.1, FB3.1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: now also C75.1
- net at C42.1, C53.1, FB1.1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: now also C76.1
- net UP_P: now reaches U2.26 (USB_DP_UP), U7.L15 (USB1_DP)
- net UP_N: now reaches U2.27 (USB_DM_UP), U7.L16 (USB1_DM)
- removed net PWR: C1.1, C24.1, C25.1, C26.1, C28.1, FB4.2, FB5.2, R6.2, R7.2, R77.1, R79.2, TP171.1, TP8.1, U20.5 (IN), U7.A7 (SYS_ADC_1P8V), U7.B7 (VREFP), U7.N13 (PMIC_MUX_IN), U9.5 (IN)
- new net 1.1V: FB4.2
- new net 1.8V: C24.1, C25.1, C26.1, TP171.1, TP8.1, U7.A7 (SYS_ADC_1P8V), U7.B7 (VREFP), U7.N13 (PMIC_MUX_IN)
- new net 5V: C1.1, C28.1, U20.5 (IN), U9.5 (IN)
Other:
- note added: "TODO: 40pf does not exist"
- note removed: "JTAG connector"
- note removed: "TODO: Series capacitance"
- note removed: "TODO: check ferrite bead location with datasheet"
