File: oresat-live-card/oresat-live-card-sch-power.kicad_sch (KiCad schematic)
At the start: 120 parts, among them Q2 PMV45EN2R, Q3 DMP2240UDM, Q4 PMV45EN2R, Q5 DMP3050LVT-7, Q6 DMP3050LVT-7, U12 MIC842LYC5, U13 MIC842LYC5, U14 MAX4211, U15 LTC3624-5, U16 MAX7310, U21 TLV73311, U22 TS5A21366, U5 LTC3624-5

Commit message: Changed to hierarchy view
updated OPD and component symbols. Resolved all DRC errors and warnings.
Parts:
- removed TP24, TP26: TEST-POINT, oresat-misc:TestPoint_Pad_D1.0mm, symbol oresat-misc:Test-Point-1mm-round
- D6, D7, D8, D9: symbol Device:LED -> Device:LED_Small_Filled
- Q3: value DMP2240UDM -> DMP2110UVTQ-7; footprint oresat-live-card:SOT23-6 -> Package_TO_SOT_SMD:SOT-23-6; DPN DMP2240UDMDICT-ND -> 31-DMP2110UVTQ-7CT-ND; MFR Diodes Incorporated -> Diodes Incorporated; MPN DMP2240UDM-7 -> DMP2110UVTQ-7
- Q5, Q6: value DMP3050LVT-7 -> DMPH2040UVTQ-7; DPN DMP3050LVT-7DICT-ND -> 31-DMPH2040UVTQ-7CT-ND; MFR Diodes Incorporated -> Diodes Incorporated; MPN DMP3050LVT-7 -> DMPH2040UVTQ-7
- R20, R22, R32, R33, R34, R35, R36, R37, R38, R39, R40, R41, R42, R43, R44, R45, R46, R47, R48, R49, R50, R51, R52, R59, R60, R63, R64, R71, R72, R75, R92, R93, R94, R95: symbol oresat-passives:R-US -> Device:R_Small_US
- R53, R56, R58, R65, R66, R67, R68, R69, R70: value 1k -> 100; footprint Resistor_SMD:R_0603_1608Metric -> oresat-passives:0603-C; symbol oresat-passives:R-US -> Device:R_Small_US; DIS (none) -> DigiKey; DPN P10.0KHCT-ND -> P100HCT-ND; MPN ERJ-3EKF1002V -> ERJ-3EKF1000V; now in the parts list
- R54, R55, R57: value 1k -> 100; symbol oresat-passives:R-US -> Device:R_Small_US; DPN P1.00KHCT-ND -> P100HCT-ND; MPN ERJ-3EKF1001V -> ERJ-3EKF1000V
- R61: value 2.7k -> 10k; symbol oresat-passives:R-US -> Device:R_Small_US
- U14: footprint oresat-live-card:QFN65P400X400X80-17T210 -> Package_DFN_QFN:QFN-16-1EP_4x4mm_P0.65mm_EP2.1x2.1mm; symbol oresat-ics:MAX4211FETE -> oresat-ics:MAX4211D/E/F
- U22: DPN 296-24304-1-ND -> 296-24304-1-ND; MFR Texas Instruments -> Texas Instruments; MPN TS5A21366DCUR -> TS5A21366DCUR
Connections:
- net UART0_Rx is gone; now on an unnamed net: U22.5 (NO2)
- net UART0_Tx is gone; now on an unnamed net: U22.1 (NO1)
- net ON/~{OFF}: now also U14.2 (IN)
- net at R92.2: no longer U22.2 (COM1)
- net at R93.2: no longer U22.6 (COM2)
- net C3-UART-Rx renamed C3-UART-RX
- net C3-UART-Tx renamed C3-UART-TX
- new net UART0_RX: U22.6 (COM2)
- new net UART0_TX: U22.2 (COM1)
