File: oresat-live-card/oresat-live-card-sch-sip-c.kicad_sch (KiCad schematic)
At the start: 29 parts, among them J7 DM3BT-DSF-PEJS, U11 TCAN330G, U3 THGBMJG8C4LBAU8, U7 OSD3358-512M-BSM

Commit message: Changed to hierarchy view
updated OPD and component symbols. Resolved all DRC errors and warnings.
Parts:
- D2, D3, D4, D5: symbol Device:LED -> Device:LED_Small_Filled
- R2, R3, R4, R5: symbol oresat-passives:R-US -> Device:R_Small_US
Connections:
- net UART0_Rx renamed UART0_RX
- net UART0_Tx renamed UART0_TX

Commit message: Schematic Update
Updated Schematic to help alleviate some of the DRC errors and warnings.
Connections:
- net UART0_RX renamed UART0_Rx
- net UART0_TX renamed UART0_Tx
Changed lines of the file:
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@@
 		)
 	)
-	(hierarchical_label "UART0_RX"
+	(hierarchical_label "UART0_Rx"
 		(shape input)
 		(at 154.94 100.33 90)
@@
 		)
 	)
-	(hierarchical_label "UART0_TX"
+	(hierarchical_label "UART0_Tx"
 		(shape input)
 		(at 157.48 100.33 90)

Commit message: Changed Footprints
Changed all passive component footprints to no silk variants. Fixed errors and warnings on library footprint mismatches
Parts:
- C10, C11, C12, C31, C5, C6, C78, C9, R2, R3, R4, R5: footprint oresat-passives:0603-C -> oresat-passives:0603-C-NOSILK
- C2, C8: footprint oresat-passives:0805-C -> oresat-passives:0805-C-NOSILK
Changed lines of the file:
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@@
 			)
 		)
-		(property "Footprint" "oresat-passives:0603-C"
+		(property "Footprint" "oresat-passives:0603-C-NOSILK"
 			(at 353.06 154.94 0)
 			(hide yes)
@@
 			)
 		)
-		(property "Footprint" "oresat-passives:0603-C"
+		(property "Footprint" "oresat-passives:0603-C-NOSILK"
 			(at 375.92 154.94 0)
 			(hide yes)
@@
 			)
 		)
-		(property "Footprint" "oresat-passives:0603-C"
+		(property "Footprint" "oresat-passives:0603-C-NOSILK"
 			(at 265.43 118.11 0)
 			(hide yes)
@@
 			)
 		)
-		(property "Footprint" "oresat-passives:0603-C"
+		(property "Footprint" "oresat-passives:0603-C-NOSILK"
 			(at 360.68 154.94 0)
 			(hide yes)
@@
 			)
 		)
-		(property "Footprint" "oresat-passives:0603-C"
+		(property "Footprint" "oresat-passives:0603-C-NOSILK"
 			(at 383.54 154.94 0)
 			(hide yes)
@@
 			)
 		)
-		(property "Footprint" "oresat-passives:0603-C"
+		(property "Footprint" "oresat-passives:0603-C-NOSILK"
 			(at 265.43 95.25 0)
 			(hide yes)
@@
 			)
 		)
-		(property "Footprint" "oresat-passives:0805-C"
+		(property "Footprint" "oresat-passives:0805-C-NOSILK"
 			(at 55.88 110.49 0)
 			(hide yes)
@@
 			)
 		)
-		(property "Footprint" "oresat-passives:0603-C"
+		(property "Footprint" "oresat-passives:0603-C-NOSILK"
 			(at 265.43 102.87 0)
 			(hide yes)
@@
 			)
 		)
-		(property "Footprint" "oresat-passives:0603-C"
+		(property "Footprint" "oresat-passives:0603-C-NOSILK"
 			(at 345.44 154.94 0)
 			(hide yes)
@@
 			)
 		)
-		(property "Footprint" "oresat-passives:0603-C"
+		(property "Footprint" "oresat-passives:0603-C-NOSILK"
 			(at 265.43 110.49 0)
 			(hide yes)
@@
 			)
 		)
-		(property "Footprint" "oresat-passives:0603-C"
+		(property "Footprint" "oresat-passives:0603-C-NOSILK"
 			(at 368.3 154.94 0)
 			(hide yes)
@@
 			)
 		)
-		(property "Footprint" "oresat-passives:0603-C"
+		(property "Footprint" "oresat-passives:0603-C-NOSILK"
 			(at 66.04 110.49 0)
 			(hide yes)
@@
 			)
 		)
-		(property "Footprint" "oresat-passives:0603-C"
+		(property "Footprint" "oresat-passives:0603-C-NOSILK"
 			(at 173.99 46.99 0)
 			(hide yes)
@@
 			)
 		)
-		(property "Footprint" "oresat-passives:0805-C"
+		(property "Footprint" "oresat-passives:0805-C-NOSILK"
 			(at 391.16 154.94 0)
 			(hide yes)
