File: oresat-live-card/oresat-live-card-sch-wifi-pa.kicad_sch (KiCad schematic)
At the start: 28 parts, among them J9 U.FL, U17 PAT1220-C-3DB, U19 TQP9111, U8 MIC94070YC6-TR

Commit message: Changed to hierarchy view
updated OPD and component symbols. Resolved all DRC errors and warnings.
Parts:
- D11: symbol Device:LED -> Device:LED_Small_Filled
- R17, R30, R80, R81, R82, R84: symbol oresat-passives:R-US -> Device:R_Small_US

Commit message: Changed Footprints
Changed all passive component footprints to no silk variants. Fixed errors and warnings on library footprint mismatches
Parts:
- C21, C43, C45, C46, C47, R17, R30, R82: footprint oresat-passives:0603-C -> oresat-passives:0603-C-NOSILK
- C48, C49, C50, C51, C52, L7, L9, R81, R84: footprint oresat-passives:0402-C -> oresat-passives:0402-C-NOSILK
- L8, R80: footprint oresat-passives:0805-C -> oresat-passives:0805-C-NOSILK
Changed lines of the file:
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@@
 			)
 		)
-		(property "Footprint" "oresat-passives:0402-C"
+		(property "Footprint" "oresat-passives:0402-C-NOSILK"
 			(at 210.82 114.3 0)
 			(hide yes)
@@
 			)
 		)
-		(property "Footprint" "oresat-passives:0603-C"
+		(property "Footprint" "oresat-passives:0603-C-NOSILK"
 			(at 247.65 199.39 0)
 			(hide yes)
@@
 			)
 		)
-		(property "Footprint" "oresat-passives:0603-C"
+		(property "Footprint" "oresat-passives:0603-C-NOSILK"
 			(at 266.7 74.93 0)
 			(hide yes)
@@
 			)
 		)
-		(property "Footprint" "oresat-passives:0603-C"
+		(property "Footprint" "oresat-passives:0603-C-NOSILK"
 			(at 219.71 74.93 0)
 			(hide yes)
@@
 			)
 		)
-		(property "Footprint" "oresat-passives:0402-C"
+		(property "Footprint" "oresat-passives:0402-C-NOSILK"
 			(at 285.75 118.11 0)
 			(hide yes)
@@
 			)
 		)
-		(property "Footprint" "oresat-passives:0603-C"
+		(property "Footprint" "oresat-passives:0603-C-NOSILK"
 			(at 266.7 149.86 0)
 			(hide yes)
@@
 			)
 		)
-		(property "Footprint" "oresat-passives:0603-C"
+		(property "Footprint" "oresat-passives:0603-C-NOSILK"
 			(at 190.5 207.01 0)
 			(hide yes)
@@
 			)
 		)
-		(property "Footprint" "oresat-passives:0402-C"
+		(property "Footprint" "oresat-passives:0402-C-NOSILK"
 			(at 233.68 74.93 0)
 			(hide yes)
@@
 			)
 		)
-		(property "Footprint" "oresat-passives:0402-C"
+		(property "Footprint" "oresat-passives:0402-C-NOSILK"
 			(at 205.74 118.11 0)
 			(hide yes)
@@
 			)
 		)
-		(property "Footprint" "oresat-passives:0805-C"
+		(property "Footprint" "oresat-passives:0805-C-NOSILK"
 			(at 247.65 81.28 0)
 			(hide yes)
@@
 			)
 		)
-		(property "Footprint" "oresat-passives:0603-C"
+		(property "Footprint" "oresat-passives:0603-C-NOSILK"
 			(at 195.58 185.42 0)
 			(hide yes)
@@
 			)
 		)
-		(property "Footprint" "oresat-passives:0402-C"
+		(property "Footprint" "oresat-passives:0402-C-NOSILK"
 			(at 254 149.86 0)
 			(hide yes)
@@
 			)
 		)
-		(property "Footprint" "oresat-passives:0402-C"
+		(property "Footprint" "oresat-passives:0402-C-NOSILK"
 			(at 294.64 114.3 0)
 			(hide yes)
@@
 			)
 		)
-		(property "Footprint" "oresat-passives:0402-C"
+		(property "Footprint" "oresat-passives:0402-C-NOSILK"
 			(at 302.26 118.11 0)
 			(hide yes)
@@
 			)
 		)
-		(property "Footprint" "oresat-passives:0603-C"
+		(property "Footprint" "oresat-passives:0603-C-NOSILK"
 			(at 278.13 74.93 0)
 			(hide yes)
@@
 			)
 		)
-		(property "Footprint" "oresat-passives:0805-C"
+		(property "Footprint" "oresat-passives:0805-C-NOSILK"
 			(at 254 57.15 0)
 			(hide yes)
@@
 			)
 		)
-		(property "Footprint" "oresat-passives:0402-C"
+		(property "Footprint" "oresat-passives:0402-C-NOSILK"
 			(at 318.77 114.3 0)
 			(hide yes)
@@
 			)
 		)
-		(property "Footprint" "oresat-passives:0402-C"
+		(property "Footprint" "oresat-passives:0402-C-NOSILK"
 			(at 223.52 114.3 0)
 			(hide yes)
@@
 			)
 		)
-		(property "Footprint" "oresat-passives:0603-C"
+		(property "Footprint" "oresat-passives:0603-C-NOSILK"
 			(at 260.35 82.55 0)
 			(hide yes)
