File: oresat-live-card/oresat-live-card-sch-wifi-switch.kicad_sch (KiCad schematic)
At the start: 43 parts, among them J11 2X1_TH_JUMPER, J15 2X1_TH_JUMPER, U24 LTC6994-1, U25 LTC6994-1, U26 SN74LVC1G32QDBVRQ1, U30 SN74LV1T34, U32 SN74LV1T34, U34 QPC1022, U35 SN74LVC1G32QDBVRQ1, U36 QPC1022, U6 SN74LVC1G04DCKR

Commit message: Changed to hierarchy view
updated OPD and component symbols. Resolved all DRC errors and warnings.
Parts:
- R103, R104, R107, R108, R114, R115, R116, R117, R122, R123, R124, R125, R86, R87: symbol Device:R_US -> Device:R_Small_US
- R16, R62: symbol oresat-passives:R-US -> Device:R_Small_US

Commit message: Changed Footprints
Changed all passive component footprints to no silk variants. Fixed errors and warnings on library footprint mismatches
Parts:
- C103, C104, C115, C116, C117, C24, C94, R116, R117, R124, R125: footprint oresat-passives:0402-C -> oresat-passives:0402-C-NOSILK
- C105, C118, C15, C86, C87, C88, C89, C98, C99, R103, R104, R107, R108, R114, R115, R122, R123, R16, R62, R86, R87: footprint oresat-passives:0603-C -> oresat-passives:0603-C-NOSILK
Changed lines of the file:
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@@
 			)
 		)
-		(property "Footprint" "oresat-passives:0603-C"
+		(property "Footprint" "oresat-passives:0603-C-NOSILK"
 			(at 160.02 73.66 0)
 			(hide yes)
@@
 			)
 		)
-		(property "Footprint" "oresat-passives:0603-C"
+		(property "Footprint" "oresat-passives:0603-C-NOSILK"
 			(at 349.25 110.49 0)
 			(hide yes)
@@
 			)
 		)
-		(property "Footprint" "oresat-passives:0402-C"
+		(property "Footprint" "oresat-passives:0402-C-NOSILK"
 			(at 264.16 204.47 0)
 			(hide yes)
@@
 			)
 		)
-		(property "Footprint" "oresat-passives:0402-C"
+		(property "Footprint" "oresat-passives:0402-C-NOSILK"
 			(at 294.64 204.47 0)
 			(hide yes)
@@
 			)
 		)
-		(property "Footprint" "oresat-passives:0402-C"
+		(property "Footprint" "oresat-passives:0402-C-NOSILK"
 			(at 337.82 229.87 0)
 			(hide yes)
@@
 			)
 		)
-		(property "Footprint" "oresat-passives:0402-C"
+		(property "Footprint" "oresat-passives:0402-C-NOSILK"
 			(at 259.08 229.87 0)
 			(hide yes)
@@
 			)
 		)
-		(property "Footprint" "oresat-passives:0603-C"
+		(property "Footprint" "oresat-passives:0603-C-NOSILK"
 			(at 340.36 190.5 0)
 			(hide yes)
@@
 			)
 		)
-		(property "Footprint" "oresat-passives:0603-C"
+		(property "Footprint" "oresat-passives:0603-C-NOSILK"
 			(at 104.14 50.8 0)
 			(hide yes)
@@
 			)
 		)
-		(property "Footprint" "oresat-passives:0603-C"
+		(property "Footprint" "oresat-passives:0603-C-NOSILK"
 			(at 128.27 158.75 0)
 			(hide yes)
@@
 			)
 		)
-		(property "Footprint" "oresat-passives:0603-C"
+		(property "Footprint" "oresat-passives:0603-C-NOSILK"
 			(at 349.25 124.46 0)
 			(hide yes)
@@
 			)
 		)
-		(property "Footprint" "oresat-passives:0603-C"
+		(property "Footprint" "oresat-passives:0603-C-NOSILK"
 			(at 66.04 39.37 0)
 			(hide yes)
@@
 			)
 		)
-		(property "Footprint" "oresat-passives:0603-C"
+		(property "Footprint" "oresat-passives:0603-C-NOSILK"
 			(at 195.58 121.92 0)
 			(hide yes)
@@
 			)
 		)
-		(property "Footprint" "oresat-passives:0603-C"
+		(property "Footprint" "oresat-passives:0603-C-NOSILK"
 			(at 288.29 73.66 0)
 			(hide yes)
@@
 			)
 		)
-		(property "Footprint" "oresat-passives:0603-C"
+		(property "Footprint" "oresat-passives:0603-C-NOSILK"
 			(at 222.25 190.5 0)
 			(hide yes)
@@
 			)
 		)
-		(property "Footprint" "oresat-passives:0402-C"
+		(property "Footprint" "oresat-passives:0402-C-NOSILK"
 			(at 302.26 229.87 0)
 			(hide yes)
@@
 			)
 		)
-		(property "Footprint" "oresat-passives:0603-C"
+		(property "Footprint" "oresat-passives:0603-C-NOSILK"
 			(at 110.49 71.12 0)
 			(hide yes)
@@
 			)
 		)
-		(property "Footprint" "oresat-passives:0603-C"
+		(property "Footprint" "oresat-passives:0603-C-NOSILK"
 			(at 325.12 48.26 0)
 			(hide yes)
@@
 			)
 		)
-		(property "Footprint" "oresat-passives:0603-C"
+		(property "Footprint" "oresat-passives:0603-C-NOSILK"
 			(at 335.28 68.58 0)
 			(hide yes)
@@
 			)
 		)
-		(property "Footprint" "oresat-passives:0402-C"
+		(property "Footprint" "oresat-passives:0402-C-NOSILK"
 			(at 264.16 194.31 0)
 			(hide yes)
@@
 			)
 		)
-		(property "Footprint" "oresat-passives:0402-C"
+		(property "Footprint" "oresat-passives:0402-C-NOSILK"
 			(at 233.68 190.5 0)
 			(hide yes)
@@
 			)
 		)
-		(property "Footprint" "oresat-passives:0603-C"
+		(property "Footprint" "oresat-passives:0603-C-NOSILK"
 			(at 207.01 154.94 0)
 			(hide yes)
@@
 			)
 		)
-		(property "Footprint" "oresat-passives:0402-C"
+		(property "Footprint" "oresat-passives:0402-C-NOSILK"
 			(at 294.64 193.04 0)
 			(hide yes)
@@
 			)
 		)
-		(property "Footprint" "oresat-passives:0603-C"
+		(property "Footprint" "oresat-passives:0603-C-NOSILK"
 			(at 266.7 99.06 0)
 			(hide yes)
@@
 			)
 		)
-		(property "Footprint" "oresat-passives:0402-C"
+		(property "Footprint" "oresat-passives:0402-C-NOSILK"
 			(at 213.36 232.41 0)
 			(hide yes)
@@
 			)
 		)
-		(property "Footprint" "oresat-passives:0603-C"
+		(property "Footprint" "oresat-passives:0603-C-NOSILK"
 			(at 140.97 100.33 0)
 			(hide yes)
@@
 			)
 		)
-		(property "Footprint" "oresat-passives:0402-C"
+		(property "Footprint" "oresat-passives:0402-C-NOSILK"
 			(at 328.93 190.5 0)
 			(hide yes)
@@
 			)
 		)
-		(property "Footprint" "oresat-passives:0603-C"
+		(property "Footprint" "oresat-passives:0603-C-NOSILK"
 			(at 147.32 129.54 0)
 			(hide yes)
@@
 			)
 		)
-		(property "Footprint" "oresat-passives:0402-C"
+		(property "Footprint" "oresat-passives:0402-C-NOSILK"
 			(at 207.01 121.92 0)
 			(hide yes)
@@
 			)
 		)
-		(property "Footprint" "oresat-passives:0603-C"
+		(property "Footprint" "oresat-passives:0603-C-NOSILK"
 			(at 67.31 76.2 0)
 			(hide yes)
@@
 			)
 		)
-		(property "Footprint" "oresat-passives:0603-C"
+		(property "Footprint" "oresat-passives:0603-C-NOSILK"
 			(at 287.02 35.56 0)
 			(hide yes)
@@
 			)
 		)
-		(property "Footprint" "oresat-passives:0603-C"
+		(property "Footprint" "oresat-passives:0603-C-NOSILK"
 			(at 43.18 101.6 0)
 			(hide yes)
@@
 			)
 		)
-		(property "Footprint" "oresat-passives:0603-C"
+		(property "Footprint" "oresat-passives:0603-C-NOSILK"
 			(at 207.01 167.64 0)
 			(hide yes)
