File: oresat-live-card/oresat-live-card-sch-usb-hub.kicad_sch (KiCad schematic)
At the start: 55 parts, among them U2 TUSB4020BI, U20 TPS2041BQDBVRQ1, U9 TPS2041BQDBVRQ1, Y3 24MHz

Commit message: Schematic Update
Updated Schematic to help alleviate some of the DRC errors and warnings.
Connections:
- net WIFI_VUSB: now also R21.1; no longer R21.2
- net at D10.2 (A): now also R21.2; no longer R21.1
Changed lines of the file:
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@@
 	)
 	(junction
+		(at 351.79 196.85)
+		(diameter 0)
+		(color 0 0 0 0)
+	)
+	(junction
 		(at 341.63 167.64)
 		(diameter 0)
@@
 	)
 	(junction
-		(at 351.79 196.85)
-		(diameter 0)
-		(color 0 0 0 0)
-	)
-	(junction
 		(at 186.69 109.22)
 		(diameter 0)
@@
 	(wire
 		(pts
-			(xy 351.79 191.77) (xy 351.79 196.85)
-		)
-		(stroke
-			(width 0)
-			(type default)
-		)
-	)
-	(wire
-		(pts
 			(xy 104.14 181.61) (xy 104.14 184.15)
 		)
@@
 	(wire
 		(pts
+			(xy 351.79 182.88) (xy 351.79 186.69)
+		)
+		(stroke
+			(width 0)
+			(type default)
+		)
+	)
+	(wire
+		(pts
 			(xy 146.05 97.79) (xy 146.05 101.6)
 		)
@@
 	(wire
 		(pts
-			(xy 361.95 196.85) (xy 351.79 196.85)
+			(xy 341.63 196.85) (xy 351.79 196.85)
 		)
 		(stroke
@@
 	(wire
 		(pts
+			(xy 351.79 196.85) (xy 361.95 196.85)
+		)
+		(stroke
+			(width 0)
+			(type default)
+		)
+	)
+	(wire
+		(pts
 			(xy 186.69 114.3) (xy 193.04 114.3)
 		)
@@
 	(wire
 		(pts
-			(xy 351.79 182.88) (xy 351.79 186.69)
-		)
-		(stroke
-			(width 0)
-			(type default)
-		)
-	)
-	(wire
-		(pts
 			(xy 93.98 114.3) (xy 100.33 114.3)
 		)
@@
 	(wire
 		(pts
+			(xy 351.79 191.77) (xy 351.79 196.85)
+		)
+		(stroke
+			(width 0)
+			(type default)
+		)
+	)
+	(wire
+		(pts
 			(xy 110.49 191.77) (xy 116.84 191.77)
 		)
@@
 	(wire
 		(pts
-			(xy 341.63 196.85) (xy 351.79 196.85)
-		)
-		(stroke
-			(width 0)
-			(type default)
-		)
-	)
-	(wire
-		(pts
 			(xy 62.23 180.34) (xy 67.31 180.34)
 		)
@@
 		(lib_id "Device:R_Small_US")
 		(at 351.79 189.23 0)
-		(mirror y)
+		(mirror x)
 		(unit 1)
 		(body_style 1)
@@
 		(dnp no)
 		(property "Reference" "R21"
-			(at 350.012 190.246 0)
+			(at 353.568 188.214 0)
 			(show_name no)
 			(do_not_autoplace no)
@@
 		)
 		(property "Value" "10k"
-			(at 349.758 192.786 0)
+			(at 353.822 185.674 0)
 			(show_name no)
 			(do_not_autoplace no)

Commit message: Changed Footprints
Changed all passive component footprints to no silk variants. Fixed errors and warnings on library footprint mismatches
Parts:
- C1, C27, C28, C42, C54, C55, C56, C57, C58, C59, C60, C63, C64, C65, C66, C67, C68, C70, C71, C72, C73, R21, R29, R6, R7, R76, R77, R78, R79, R83, R89, R90, R91, R98, R99: footprint oresat-passives:0603-C -> oresat-passives:0603-C-NOSILK
- C53, C69, C76, C96, C97: footprint oresat-passives:0805-C -> oresat-passives:0805-C-NOSILK
Changed lines of the file:
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@@
 			)
 		)
-		(property "Footprint" "oresat-passives:0603-C"
+		(property "Footprint" "oresat-passives:0603-C-NOSILK"
 			(at 236.22 160.02 0)
 			(hide yes)
@@
 			)
 		)
-		(property "Footprint" "oresat-passives:0603-C"
+		(property "Footprint" "oresat-passives:0603-C-NOSILK"
 			(at 59.69 180.34 0)
 			(hide yes)
@@
 			)
 		)
-		(property "Footprint" "oresat-passives:0603-C"
+		(property "Footprint" "oresat-passives:0603-C-NOSILK"
 			(at 180.34 111.76 0)
 			(hide yes)
@@
 			)
 		)
-		(property "Footprint" "oresat-passives:0805-C"
+		(property "Footprint" "oresat-passives:0805-C-NOSILK"
 			(at 294.64 97.79 0)
 			(hide yes)
@@
 			)
 		)
-		(property "Footprint" "oresat-passives:0805-C"
+		(property "Footprint" "oresat-passives:0805-C-NOSILK"
 			(at 284.48 172.72 0)
 			(hide yes)
@@
 			)
 		)
-		(property "Footprint" "oresat-passives:0603-C"
+		(property "Footprint" "oresat-passives:0603-C-NOSILK"
 			(at 59.69 160.02 0)
 			(hide yes)
@@
 			)
 		)
-		(property "Footprint" "oresat-passives:0603-C"
+		(property "Footprint" "oresat-passives:0603-C-NOSILK"
 			(at 154.94 111.76 0)
 			(hide yes)
@@
 			)
 		)
-		(property "Footprint" "oresat-passives:0603-C"
+		(property "Footprint" "oresat-passives:0603-C-NOSILK"
 			(at 119.38 111.76 0)
 			(hide yes)
@@
 			)
 		)
-		(property "Footprint" "oresat-passives:0805-C"
+		(property "Footprint" "oresat-passives:0805-C-NOSILK"
 			(at 294.64 172.72 0)
 			(hide yes)
@@
 			)
 		)
-		(property "Footprint" "oresat-passives:0603-C"
+		(property "Footprint" "oresat-passives:0603-C-NOSILK"
 			(at 274.32 172.72 0)
 			(hide yes)
@@
 			)
 		)
-		(property "Footprint" "oresat-passives:0805-C"
+		(property "Footprint" "oresat-passives:0805-C-NOSILK"
 			(at 284.48 97.79 0)
 			(hide yes)
@@
 			)
 		)
-		(property "Footprint" "oresat-passives:0603-C"
+		(property "Footprint" "oresat-passives:0603-C-NOSILK"
 			(at 351.79 189.23 0)
 			(hide yes)
@@
 			)
 		)
-		(property "Footprint" "oresat-passives:0603-C"
+		(property "Footprint" "oresat-passives:0603-C-NOSILK"
 			(at 173.99 111.76 0)
 			(hide yes)
@@
 			)
 		)
-		(property "Footprint" "oresat-passives:0603-C"
+		(property "Footprint" "oresat-passives:0603-C-NOSILK"
 			(at 200.66 111.76 0)
 			(hide yes)
@@
 			)
 		)
-		(property "Footprint" "oresat-passives:0603-C"
+		(property "Footprint" "oresat-passives:0603-C-NOSILK"
 			(at 238.76 85.09 0)
 			(hide yes)
@@
 			)
 		)
-		(property "Footprint" "oresat-passives:0603-C"
+		(property "Footprint" "oresat-passives:0603-C-NOSILK"
 			(at 106.68 111.76 0)
 			(hide yes)
@@
 			)
 		)
-		(property "Footprint" "oresat-passives:0603-C"
+		(property "Footprint" "oresat-passives:0603-C-NOSILK"
 			(at 100.33 111.76 0)
 			(hide yes)
@@
 			)
 		)
-		(property "Footprint" "oresat-passives:0603-C"
+		(property "Footprint" "oresat-passives:0603-C-NOSILK"
 			(at 113.03 111.76 0)
 			(hide yes)
@@
 			)
 		)
-		(property "Footprint" "oresat-passives:0603-C"
+		(property "Footprint" "oresat-passives:0603-C-NOSILK"
 			(at 77.47 129.54 0)
 			(hide yes)
@@
 			)
 		)
-		(property "Footprint" "oresat-passives:0603-C"
+		(property "Footprint" "oresat-passives:0603-C-NOSILK"
 			(at 264.16 151.13 0)
 			(hide yes)
@@
 			)
 		)
-		(property "Footprint" "oresat-passives:0603-C"
+		(property "Footprint" "oresat-passives:0603-C-NOSILK"
 			(at 193.04 111.76 0)
 			(hide yes)
@@
 			)
 		)
-		(property "Footprint" "oresat-passives:0603-C"
+		(property "Footprint" "oresat-passives:0603-C-NOSILK"
 			(at 233.68 85.09 0)
 			(hide yes)
@@
 			)
 		)
-		(property "Footprint" "oresat-passives:0603-C"
+		(property "Footprint" "oresat-passives:0603-C-NOSILK"
 			(at 107.95 152.4 0)
 			(hide yes)
@@
 			)
 		)
-		(property "Footprint" "oresat-passives:0603-C"
+		(property "Footprint" "oresat-passives:0603-C-NOSILK"
 			(at 264.16 76.2 0)
 			(hide yes)
@@
 			)
 		)
-		(property "Footprint" "oresat-passives:0603-C"
+		(property "Footprint" "oresat-passives:0603-C-NOSILK"
 			(at 148.59 111.76 0)
 			(hide yes)
@@
 			)
 		)
-		(property "Footprint" "oresat-passives:0603-C"
+		(property "Footprint" "oresat-passives:0603-C-NOSILK"
 			(at 161.29 111.76 0)
 			(hide yes)
@@
 			)
 		)
-		(property "Footprint" "oresat-passives:0603-C"
+		(property "Footprint" "oresat-passives:0603-C-NOSILK"
 			(at 104.14 186.69 0)
 			(hide yes)
@@
 			)
 		)
-		(property "Footprint" "oresat-passives:0805-C"
+		(property "Footprint" "oresat-passives:0805-C-NOSILK"
 			(at 132.08 111.76 0)
 			(hide yes)
@@
 			)
 		)
-		(property "Footprint" "oresat-passives:0603-C"
+		(property "Footprint" "oresat-passives:0603-C-NOSILK"
 			(at 241.3 160.02 0)
 			(hide yes)
@@
 			)
 		)
-		(property "Footprint" "oresat-passives:0603-C"
+		(property "Footprint" "oresat-passives:0603-C-NOSILK"
 			(at 167.64 111.76 0)
 			(hide yes)
@@
 			)
 		)
-		(property "Footprint" "oresat-passives:0603-C"
+		(property "Footprint" "oresat-passives:0603-C-NOSILK"
 			(at 256.54 140.97 0)
 			(hide yes)
@@
 			)
 		)
-		(property "Footprint" "oresat-passives:0603-C"
+		(property "Footprint" "oresat-passives:0603-C-NOSILK"
 			(at 125.73 111.76 0)
 			(hide yes)
@@
 			)
 		)
-		(property "Footprint" "oresat-passives:0603-C"
+		(property "Footprint" "oresat-passives:0603-C-NOSILK"
 			(at 361.95 189.23 0)
 			(hide yes)
@@
 			)
 		)
-		(property "Footprint" "oresat-passives:0603-C"
+		(property "Footprint" "oresat-passives:0603-C-NOSILK"
 			(at 99.06 179.07 0)
 			(hide yes)
@@
 			)
 		)
-		(property "Footprint" "oresat-passives:0603-C"
+		(property "Footprint" "oresat-passives:0603-C-NOSILK"
 			(at 274.32 97.79 0)
 			(hide yes)
@@
 			)
 		)
-		(property "Footprint" "oresat-passives:0603-C"
+		(property "Footprint" "oresat-passives:0603-C-NOSILK"
 			(at 77.47 142.24 0)
 			(hide yes)
@@
 			)
 		)
-		(property "Footprint" "oresat-passives:0603-C"
+		(property "Footprint" "oresat-passives:0603-C-NOSILK"
 			(at 93.98 111.76 0)
 			(hide yes)
@@
 			)
 		)
-		(property "Footprint" "oresat-passives:0603-C"
+		(property "Footprint" "oresat-passives:0603-C-NOSILK"
 			(at 256.54 66.04 0)
 			(hide yes)
@@
 			)
 		)
-		(property "Footprint" "oresat-passives:0603-C"
+		(property "Footprint" "oresat-passives:0603-C-NOSILK"
 			(at 186.69 111.76 0)
 			(hide yes)
@@
 			)
 		)
-		(property "Footprint" "oresat-passives:0603-C"
+		(property "Footprint" "oresat-passives:0603-C-NOSILK"
 			(at 88.9 142.24 0)
 			(hide yes)

Commit message: Schematic and PCB update
updated hierarchy labels to have more clarifying names. Fixed RF connector symbol to footprint issues. Linked footprints and 3d models. Added DRC error clearance to ignore of specific RF class. Fixed most of all the DRC warnings and errors outside emmc and silkscreen on exposed copper
Changed lines of the file:
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@@
 	)
 	(hierarchical_label "WIFI_USB_N"
-		(shape output)
+		(shape bidirectional)
 		(at 364.49 170.18 0)
 		(effects
@@
 	)
 	(hierarchical_label "CAMERA_USB_P"
-		(shape output)
+		(shape bidirectional)
 		(at 361.95 115.57 0)
 		(effects
@@
 	)
 	(hierarchical_label "UP_N"
-		(shape input)
+		(shape bidirectional)
 		(at 104.14 130.81 180)
 		(effects
@@
 	)
 	(hierarchical_label "CAMERA_USB_N"
-		(shape output)
+		(shape bidirectional)
 		(at 361.95 118.11 0)
 		(effects
@@
 	)
 	(hierarchical_label "WIFI_USB_P"
-		(shape output)
+		(shape bidirectional)
 		(at 364.49 172.72 0)
 		(effects
@@
 	)
 	(hierarchical_label "UP_P"
-		(shape input)
+		(shape bidirectional)
 		(at 104.14 128.27 180)
 		(effects

Commit message: First commit
Parts:
- C1, C27, C28, C42, C54, C55, C56, C57, C58, C59, C60, C63, C64, C65, C66, C67, C68, C70, C71, C72, C73: footprint oresat-passives:0603-C-NOSILK -> oresat-passives:0603-C
- C53, C69, C76, C96, C97: footprint oresat-passives:0805-C-NOSILK -> oresat-passives:0805-C
- R78: value 9.53k -> 0; footprint oresat-passives:0603-C-NOSILK -> oresat-passives:0805-C; DPN P9.53KHCT-ND -> P0.0ACT-ND; MPN ERJ-3EKF9531V -> ERJ-6GEY0R00V
- R83: value 90.9k -> 3.3; footprint oresat-passives:0603-C-NOSILK -> oresat-passives:0402-C; DPN P90.9KHCT-ND -> 541-3.30LLCT-ND; MFR Panasonic -> Vishay Dale; MPN ERJ-3EKF9092V -> CRCW04023R30FKED
Changed lines of the file:
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@@
 			)
 		)
-		(property "Footprint" "oresat-passives:0603-C-NOSILK"
+		(property "Footprint" "oresat-passives:0603-C"
 			(at 59.69 180.34 0)
 			(hide yes)
@@
 			)
 		)
-		(property "Footprint" "oresat-passives:0603-C-NOSILK"
+		(property "Footprint" "oresat-passives:0603-C"
 			(at 180.34 111.76 0)
 			(hide yes)
@@
 			)
 		)
-		(property "Footprint" "oresat-passives:0805-C-NOSILK"
+		(property "Footprint" "oresat-passives:0805-C"
 			(at 294.64 97.79 0)
 			(hide yes)
@@
 			)
 		)
-		(property "Footprint" "oresat-passives:0805-C-NOSILK"
+		(property "Footprint" "oresat-passives:0805-C"
 			(at 284.48 172.72 0)
 			(hide yes)
@@
 			)
 		)
-		(property "Footprint" "oresat-passives:0603-C-NOSILK"
+		(property "Footprint" "oresat-passives:0603-C"
 			(at 59.69 160.02 0)
 			(hide yes)
@@
 			)
 		)
-		(property "Footprint" "oresat-passives:0603-C-NOSILK"
+		(property "Footprint" "oresat-passives:0603-C"
 			(at 154.94 111.76 0)
 			(hide yes)
@@
 			)
 		)
-		(property "Footprint" "oresat-passives:0603-C-NOSILK"
+		(property "Footprint" "oresat-passives:0603-C"
 			(at 119.38 111.76 0)
 			(hide yes)
@@
 			)
 		)
-		(property "Footprint" "oresat-passives:0805-C-NOSILK"
+		(property "Footprint" "oresat-passives:0805-C"
 			(at 294.64 172.72 0)
 			(hide yes)
@@
 			)
 		)
-		(property "Footprint" "oresat-passives:0603-C-NOSILK"
+		(property "Footprint" "oresat-passives:0603-C"
 			(at 274.32 172.72 0)
 			(hide yes)
@@
 			)
 		)
-		(property "Footprint" "oresat-passives:0805-C-NOSILK"
+		(property "Footprint" "oresat-passives:0805-C"
 			(at 284.48 97.79 0)
 			(hide yes)
@@
 			)
 		)
-		(property "Footprint" "oresat-passives:0603-C-NOSILK"
+		(property "Footprint" "oresat-passives:0603-C"
 			(at 173.99 111.76 0)
 			(hide yes)
@@
 			)
 		)
-		(property "Footprint" "oresat-passives:0603-C-NOSILK"
+		(property "Footprint" "oresat-passives:0603-C"
 			(at 200.66 111.76 0)
 			(hide yes)
@@
 			)
 		)
-		(property "Footprint" "oresat-passives:0603-C-NOSILK"
+		(property "Footprint" "oresat-passives:0603-C"
 			(at 106.68 111.76 0)
 			(hide yes)
@@
 			)
 		)
-		(property "Footprint" "oresat-passives:0603-C-NOSILK"
+		(property "Footprint" "oresat-passives:0603-C"
 			(at 100.33 111.76 0)
 			(hide yes)
@@
 			)
 		)
-		(property "Footprint" "oresat-passives:0603-C-NOSILK"
+		(property "Footprint" "oresat-passives:0603-C"
 			(at 113.03 111.76 0)
 			(hide yes)
@@
 			)
 		)
-		(property "Value" "90.9k"
+		(property "Value" "3.3"
 			(at 78.486 129.286 0)
 			(show_name no)
@@
 			)
 		)
-		(property "Footprint" "oresat-passives:0603-C-NOSILK"
+		(property "Footprint" "oresat-passives:0402-C"
 			(at 77.47 129.54 0)
 			(hide yes)
@@
 			)
 		)
-		(property "Description" "Resistor, small US symbol"
+		(property "Description" "RES SMD 3.3 OHM 1% 1/16W 0402"
 			(at 77.47 129.54 0)
 			(hide yes)
@@
 			)
 		)
-		(property "MPN" "ERJ-3EKF9092V"
+		(property "MPN" "CRCW04023R30FKED"
 			(at 77.47 129.54 0)
 			(hide yes)
@@
 			)
 		)
-		(property "DPN" "P90.9KHCT-ND "
+		(property "DPN" "541-3.30LLCT-ND "
 			(at 77.47 129.54 90)
 			(hide yes)
@@
 			)
 		)
-		(property "MFR" "Panasonic "
+		(property "MFR" "Vishay Dale "
 			(at 77.47 129.54 90)
 			(hide yes)
@@
 			)
 		)
-		(property "Footprint" "oresat-passives:0603-C-NOSILK"
+		(property "Footprint" "oresat-passives:0603-C"
 			(at 264.16 151.13 0)
 			(hide yes)
@@
 			)
 		)
-		(property "Footprint" "oresat-passives:0603-C-NOSILK"
+		(property "Footprint" "oresat-passives:0603-C"
 			(at 193.04 111.76 0)
 			(hide yes)
@@
 			)
 		)
-		(property "Footprint" "oresat-passives:0603-C-NOSILK"
+		(property "Footprint" "oresat-passives:0603-C"
 			(at 264.16 76.2 0)
 			(hide yes)
@@
 			)
 		)
-		(property "Footprint" "oresat-passives:0603-C-NOSILK"
+		(property "Footprint" "oresat-passives:0603-C"
 			(at 148.59 111.76 0)
 			(hide yes)
@@
 			)
 		)
-		(property "Footprint" "oresat-passives:0603-C-NOSILK"
+		(property "Footprint" "oresat-passives:0603-C"
 			(at 161.29 111.76 0)
 			(hide yes)
@@
 			)
 		)
-		(property "Footprint" "oresat-passives:0805-C-NOSILK"
+		(property "Footprint" "oresat-passives:0805-C"
 			(at 132.08 111.76 0)
 			(hide yes)
@@
 			)
 		)
-		(property "Footprint" "oresat-passives:0603-C-NOSILK"
+		(property "Footprint" "oresat-passives:0603-C"
 			(at 167.64 111.76 0)
 			(hide yes)
@@
 			)
 		)
-		(property "Footprint" "oresat-passives:0603-C-NOSILK"
+		(property "Footprint" "oresat-passives:0603-C"
 			(at 125.73 111.76 0)
 			(hide yes)
@@
 			)
 		)
-		(property "Footprint" "oresat-passives:0603-C-NOSILK"
+		(property "Footprint" "oresat-passives:0603-C"
 			(at 274.32 97.79 0)
 			(hide yes)
@@
 			)
 		)
-		(property "Footprint" "oresat-passives:0603-C-NOSILK"
+		(property "Footprint" "oresat-passives:0603-C"
 			(at 93.98 111.76 0)
 			(hide yes)
@@
 			)
 		)
-		(property "Description" "Light emitting diode, small symbol, filled shape"
+		(property "Description" "Green 525nm LED 3.2V 0603"
 			(at 351.79 180.34 0)
 			(hide yes)
@@
 			)
 		)
-		(property "Footprint" "oresat-passives:0603-C-NOSILK"
+		(property "Footprint" "oresat-passives:0603-C"
 			(at 186.69 111.76 0)
 			(hide yes)
@@
 			)
 		)
-		(property "Value" "9.53k"
+		(property "Value" "0"
 			(at 96.774 143.256 0)
 			(show_name no)
@@
 			)
 		)
-		(property "Footprint" "oresat-passives:0603-C-NOSILK"
+		(property "Footprint" "oresat-passives:0805-C"
 			(at 88.9 142.24 0)
 			(hide yes)
@@
 			)
 		)
-		(property "Description" "Resistor, small US symbol"
+		(property "Description" "RES SMD 0 OHM JUMPER 1/8W 0805"
 			(at 88.9 142.24 0)
 			(hide yes)
@@
 			)
 		)
-		(property "MPN" "ERJ-3EKF9531V "
+		(property "MPN" "ERJ-6GEY0R00V"
 			(at 88.9 142.24 0)
 			(hide yes)
@@
 			)
 		)
-		(property "DPN" "P9.53KHCT-ND "
+		(property "DPN" "P0.0ACT-ND "
 			(at 88.9 142.24 0)
 			(hide yes)
