File: oresat-live-card/oresat-live-card-sch-wifi-lna.kicad_sch (KiCad schematic)
At the start: 34 parts, among them J12 U.FL, J14 Conn_01x02, U18 TQP3M9037, U27 PAT1220-C-3DB, U28 PD2328J5050S2HF, U29 LTC5538

Commit message: Changed to hierarchy view
updated OPD and component symbols. Resolved all DRC errors and warnings.
Parts:
- D15: symbol Device:LED -> Device:LED_Small_Filled
- R105, R106, R109, R118, R119, R120, R121, R88: symbol Device:R_US -> Device:R_Small_US
- R85: symbol oresat-passives:R-US -> Device:R_Small_US
Other:
- moved on the sheet: C106, C107, C108, C109, C110, C111, C112, C113, C114, C90, C91, C92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

Commit message: Changed Footprints
Changed all passive component footprints to no silk variants. Fixed errors and warnings on library footprint mismatches
Parts:
- C106, C111, R105, R109, R118, R119, R120, R121, R85, R88: footprint oresat-passives:0603-C -> oresat-passives:0603-C-NOSILK
- C107, C108, C109, C110, C112, C113, C114, C90, C91, C92, C93, L4, R106: footprint oresat-passives:0402-C -> oresat-passives:0402-C-NOSILK
Changed lines of the file:
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@@
 			)
 		)
-		(property "Footprint" "oresat-passives:0402-C"
+		(property "Footprint" "oresat-passives:0402-C-NOSILK"
 			(at 312.42 134.62 0)
 			(hide yes)
@@
 			)
 		)
-		(property "Footprint" "oresat-passives:0402-C"
+		(property "Footprint" "oresat-passives:0402-C-NOSILK"
 			(at 339.09 190.5 0)
 			(hide yes)
@@
 			)
 		)
-		(property "Footprint" "oresat-passives:0603-C"
+		(property "Footprint" "oresat-passives:0603-C-NOSILK"
 			(at 67.31 154.94 0)
 			(hide yes)
@@
 			)
 		)
-		(property "Footprint" "oresat-passives:0402-C"
+		(property "Footprint" "oresat-passives:0402-C-NOSILK"
 			(at 327.66 185.42 0)
 			(hide yes)
@@
 			)
 		)
-		(property "Footprint" "oresat-passives:0603-C"
+		(property "Footprint" "oresat-passives:0603-C-NOSILK"
 			(at 370.84 165.1 0)
 			(hide yes)
@@
 			)
 		)
-		(property "Footprint" "oresat-passives:0402-C"
+		(property "Footprint" "oresat-passives:0402-C-NOSILK"
 			(at 139.7 90.17 0)
 			(hide yes)
@@
 			)
 		)
-		(property "Footprint" "oresat-passives:0402-C"
+		(property "Footprint" "oresat-passives:0402-C-NOSILK"
 			(at 246.38 181.61 0)
 			(hide yes)
@@
 			)
 		)
-		(property "Footprint" "oresat-passives:0603-C"
+		(property "Footprint" "oresat-passives:0603-C-NOSILK"
 			(at 259.08 182.88 0)
 			(hide yes)
@@
 			)
 		)
-		(property "Footprint" "oresat-passives:0603-C"
+		(property "Footprint" "oresat-passives:0603-C-NOSILK"
 			(at 81.28 148.59 0)
 			(hide yes)
@@
 			)
 		)
-		(property "Footprint" "oresat-passives:0402-C"
+		(property "Footprint" "oresat-passives:0402-C-NOSILK"
 			(at 267.97 172.72 0)
 			(hide yes)
@@
 			)
 		)
-		(property "Footprint" "oresat-passives:0402-C"
+		(property "Footprint" "oresat-passives:0402-C-NOSILK"
 			(at 279.4 184.15 0)
 			(hide yes)
@@
 			)
 		)
-		(property "Footprint" "oresat-passives:0603-C"
+		(property "Footprint" "oresat-passives:0603-C-NOSILK"
 			(at 346.71 156.21 0)
 			(hide yes)
@@
 			)
 		)
-		(property "Footprint" "oresat-passives:0603-C"
+		(property "Footprint" "oresat-passives:0603-C-NOSILK"
 			(at 88.9 157.48 0)
 			(hide yes)
@@
 			)
 		)
-		(property "Footprint" "oresat-passives:0402-C"
+		(property "Footprint" "oresat-passives:0402-C-NOSILK"
 			(at 83.82 111.76 0)
 			(hide yes)
@@
 			)
 		)
-		(property "Footprint" "oresat-passives:0402-C"
+		(property "Footprint" "oresat-passives:0402-C-NOSILK"
 			(at 252.73 172.72 0)
 			(hide yes)
@@
 			)
 		)
-		(property "Footprint" "oresat-passives:0402-C"
+		(property "Footprint" "oresat-passives:0402-C-NOSILK"
 			(at 151.13 90.17 0)
 			(hide yes)
@@
 			)
 		)
-		(property "Footprint" "oresat-passives:0402-C"
+		(property "Footprint" "oresat-passives:0402-C-NOSILK"
 			(at 137.16 111.76 0)
 			(hide yes)
@@
 			)
 		)
-		(property "Footprint" "oresat-passives:0402-C"
+		(property "Footprint" "oresat-passives:0402-C-NOSILK"
 			(at 327.66 172.72 0)
 			(hide yes)
@@
 			)
 		)
-		(property "Footprint" "oresat-passives:0603-C"
+		(property "Footprint" "oresat-passives:0603-C-NOSILK"
 			(at 312.42 144.78 0)
 			(hide yes)
@@
 			)
 		)
-		(property "Footprint" "oresat-passives:0603-C"
+		(property "Footprint" "oresat-passives:0603-C-NOSILK"
 			(at 279.4 160.02 0)
 			(hide yes)
@@
 			)
 		)
-		(property "Footprint" "oresat-passives:0603-C"
+		(property "Footprint" "oresat-passives:0603-C-NOSILK"
 			(at 246.38 114.3 0)
 			(hide yes)
@@
 			)
 		)
-		(property "Footprint" "oresat-passives:0603-C"
+		(property "Footprint" "oresat-passives:0603-C-NOSILK"
 			(at 358.14 165.1 0)
 			(hide yes)
@@
 			)
 		)
-		(property "Footprint" "oresat-passives:0402-C"
+		(property "Footprint" "oresat-passives:0402-C-NOSILK"
 			(at 129.54 81.28 0)
 			(hide yes)

Commit message: Organizational changes
Updated hierarchical labels and other misc schematic fixes
Parts:
- removed J12: U.FL, Connector_Coaxial:U.FL_Molex_MCRF_73412-0110_Vertical, symbol Connector:Conn_Coaxial
- removed PCBA1B1: WF-NP9202WF, symbol oresat-pcbs:WF-NP9202WF
Connections:
- net RF_DET_IN: now reaches R121.1, U28.4 (OUTPUT1)
Other:
- note added: "RF Detector, transforms RF detected into a DC sense line for Octavo to read"
- note removed: "Add datasheet???"
- note removed: "Connection to J12 U.FL to U.FL coax 90 - 100 mm long E.g., TE 2118651-6"
- note removed: "Same PCBA1 for TX"

Commit message: Schematic and PCB update
updated hierarchy labels to have more clarifying names. Fixed RF connector symbol to footprint issues. Linked footprints and 3d models. Added DRC error clearance to ignore of specific RF class. Fixed most of all the DRC warnings and errors outside emmc and silkscreen on exposed copper
Connections:
- net PA_ON_LNA_OFF renamed LNA_SHUTDOWN
- net RX_DET_OUT renamed RF/RX_IN_DETECTED
Changed lines of the file:
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@@
 		)
 	)
-	(hierarchical_label "PA_ON_LNA_OFF"
+	(hierarchical_label "LNA_SHUTDOWN"
 		(shape input)
 		(at 59.69 148.59 180)
@@
 		)
 	)
-	(hierarchical_label "RX_DET_OUT"
+	(hierarchical_label "RF{slash}RX_IN_DETECTED"
 		(shape output)
 		(at 391.16 156.21 0)

Commit message: First commit
Parts:
- C106, C111, R105, R109, R118, R119, R120: footprint oresat-passives:0603-C-NOSILK -> oresat-passives:0603-C
- C107, C108, C109, C110, C112, C113, C114, C90, C91, C92, C93, L4, R106: footprint oresat-passives:0402-C-NOSILK -> oresat-passives:0402-C
- L3: DIS DigiKey -> Mouser; DPN 2457-0603DC-18NXJRW-ND -> 994-0603DC-18NXJRW
Changed lines of the file:
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@@
 			)
 		)
-		(property "Footprint" "oresat-passives:0402-C-NOSILK"
+		(property "Footprint" "oresat-passives:0402-C"
 			(at 312.42 134.62 0)
 			(hide yes)
@@
 			)
 		)
-		(property "Footprint" "oresat-passives:0402-C-NOSILK"
+		(property "Footprint" "oresat-passives:0402-C"
 			(at 339.09 190.5 0)
 			(hide yes)
@@
 			)
 		)
-		(property "Footprint" "oresat-passives:0402-C-NOSILK"
+		(property "Footprint" "oresat-passives:0402-C"
 			(at 327.66 185.42 0)
 			(hide yes)
@@
 			)
 		)
-		(property "Footprint" "oresat-passives:0603-C-NOSILK"
+		(property "Footprint" "oresat-passives:0603-C"
 			(at 370.84 165.1 0)
 			(hide yes)
@@
 			)
 		)
-		(property "Description" "Light emitting diode, small symbol, filled shape"
+		(property "Description" "Green 525nm LED 3.2V 0603"
 			(at 67.31 165.1 0)
 			(hide yes)
@@
 			)
 		)
-		(property "Footprint" "oresat-passives:0402-C-NOSILK"
+		(property "Footprint" "oresat-passives:0402-C"
 			(at 139.7 90.17 0)
 			(hide yes)
@@
 			)
 		)
-		(property "Footprint" "oresat-passives:0402-C-NOSILK"
+		(property "Footprint" "oresat-passives:0402-C"
 			(at 246.38 181.61 0)
 			(hide yes)
@@
 			)
 		)
-		(property "Footprint" "oresat-passives:0603-C-NOSILK"
+		(property "Footprint" "oresat-passives:0603-C"
 			(at 259.08 182.88 0)
 			(hide yes)
@@
 			)
 		)
-		(property "Description" "Resistor, small US symbol"
+		(property "Description" "RES SMD 56 OHM 1% 1/10W 0603"
 			(at 259.08 182.88 0)
 			(hide yes)
@@
 			)
 		)
-		(property "Footprint" "oresat-passives:0603-C-NOSILK"
+		(property "Footprint" "oresat-passives:0603-C"
 			(at 81.28 148.59 0)
 			(hide yes)
@@
 			)
 		)
-		(property "Description" "Resistor, small US symbol"
+		(property "Description" "RES 33K OHM 1% 1/10W 0603"
 			(at 81.28 148.59 0)
 			(hide yes)
@@
 			)
 		)
-		(property "Footprint" "oresat-passives:0402-C-NOSILK"
+		(property "Footprint" "oresat-passives:0402-C"
 			(at 267.97 172.72 0)
 			(hide yes)
@@
 			)
 		)
-		(property "DPN" "2457-0603DC-18NXJRW-ND"
+		(property "DPN" "994-0603DC-18NXJRW  "
 			(at 129.54 95.25 0)
 			(hide yes)
@@
 			)
 		)
-		(property "DIS" "DigiKey"
+		(property "DIS" "Mouser "
 			(at 129.54 95.25 0)
 			(hide yes)
@@
 			)
 		)
-		(property "Footprint" "oresat-passives:0402-C-NOSILK"
+		(property "Footprint" "oresat-passives:0402-C"
 			(at 279.4 184.15 0)
 			(hide yes)
@@
 			)
 		)
-		(property "Footprint" "oresat-passives:0603-C-NOSILK"
+		(property "Footprint" "oresat-passives:0603-C"
 			(at 346.71 156.21 0)
 			(hide yes)
@@
 			)
 		)
-		(property "Description" "Resistor, small US symbol"
+		(property "Description" "RES SMD 4.99K OHM 1% 1/10W 0603"
 			(at 346.71 156.21 0)
 			(hide yes)
@@
 			)
 		)
-		(property "Footprint" "oresat-passives:0402-C-NOSILK"
+		(property "Footprint" "oresat-passives:0402-C"
 			(at 83.82 111.76 0)
 			(hide yes)
@@
 			)
 		)
-		(property "Footprint" "oresat-passives:0402-C-NOSILK"
+		(property "Footprint" "oresat-passives:0402-C"
 			(at 252.73 172.72 0)
 			(hide yes)
@@
 			)
 		)
-		(property "Footprint" "oresat-passives:0402-C-NOSILK"
+		(property "Footprint" "oresat-passives:0402-C"
 			(at 151.13 90.17 0)
 			(hide yes)
@@
 			)
 		)
-		(property "Footprint" "oresat-passives:0402-C-NOSILK"
+		(property "Footprint" "oresat-passives:0402-C"
 			(at 137.16 111.76 0)
 			(hide yes)
@@
 			)
 		)
-		(property "Footprint" "oresat-passives:0402-C-NOSILK"
+		(property "Footprint" "oresat-passives:0402-C"
 			(at 327.66 172.72 0)
 			(hide yes)
@@
 			)
 		)
-		(property "Footprint" "oresat-passives:0603-C-NOSILK"
+		(property "Footprint" "oresat-passives:0603-C"
 			(at 312.42 144.78 0)
 			(hide yes)
@@
 			)
 		)
-		(property "Footprint" "oresat-passives:0603-C-NOSILK"
+		(property "Footprint" "oresat-passives:0603-C"
 			(at 279.4 160.02 0)
 			(hide yes)
@@
 			)
 		)
-		(property "Description" "Resistor, small US symbol"
+		(property "Description" "RES SMD 4.99K OHM 1% 1/10W 0603"
 			(at 279.4 160.02 0)
 			(hide yes)
@@
 			)
 		)
-		(property "Footprint" "oresat-passives:0603-C-NOSILK"
+		(property "Footprint" "oresat-passives:0603-C"
 			(at 358.14 165.1 0)
 			(hide yes)
@@
 			)
 		)
-		(property "Description" "Resistor, small US symbol"
+		(property "Description" "RES SMD 4.99K OHM 1% 1/10W 0603"
 			(at 358.14 165.1 0)
 			(hide yes)
@@
 			)
 		)
-		(property "Footprint" "oresat-passives:0402-C-NOSILK"
+		(property "Footprint" "oresat-passives:0402-C"
 			(at 129.54 81.28 0)
 			(hide yes)
@@
 			)
 		)
-		(property "Description" "Resistor, small US symbol"
+		(property "Description" "RES SMD 0 OHM JUMPER 1/10W 0402"
 			(at 129.54 81.28 0)
 			(hide yes)
