File: oresat-live-card/oresat-live-card.kicad_pcb (KiCad board)
At the start: 4 copper layers, 99.8 x 94.6 mm, 379 parts, among them J1 SM14B-SHLS-TF, J10 SM06B-SRSS-TB, J11 2X1_TH_JUMPER, J12 U.FL, J14 Conn_01x02, J15 2X1_TH_JUMPER, J2 SM06B-SRSS-TB, J3 Conn_01x02, J4 TFM-120-01-L-D-RA, J5 GRPB041VWVN-RC, J6 SMPM, J7 DM3BT-DSF-PEJS, J8 SMPM, J9 U.FL, Q1 MMBT2907, Q2 DMN2050LQ-7, Q3 DMP2110UVTQ-7, Q4 DMN2050LQ-7, Q5 DMPH2040UVTQ-7, Q6 DMPH2040UVTQ-7, U10 TLVH431, U11 TCAN330G, U12 MIC842LYC5, U13 MIC842LYC5, U14 MAX4211, U15 LTC3624-5, U16 MAX7310, U17 PAT1220-C-3DB, U18 TQP3M9037, U19 TQP9111, U2 TUSB4020BI, U20 TPS2041BQDBVRQ1, U21 TLV73311, U22 TS5A21366, U23 RCLAMP0504FB, U24 LTC6994-1, U25 LTC6994-1, U26 SN74LVC1G32QDBVRQ1, U27 PAT1220-C-3DB, U28 PD2328J5050S2HF, U29 LTC5538, U3 THGBMJG8C4LBAU8, U30 SN74LV1T34, U32 SN74LV1T34, U34 QPC1022, U35 SN74LVC1G32QDBVRQ1, U36 QPC1022, U4 SN74AUC1G07DCKR, U5 LTC3624-5, U6 SN74LVC1G04DCKR, U7 OSD3358-512M-BSM, U8 MIC94070YC6-TR, U9 TPS2041BQDBVRQ1, Y1 24MHz, Y2 32.768KHZ, Y3 24MHz

Commit message: Very minor layout changes
Parts:
- moved D6 0.33 mm to (112.8, 73.8)
- moved R49 0.33 mm to (116.0, 73.8)
- moved C31 0.26 mm to (112.5, 75.9), turned to -90 degrees
Routing:
- net +3.3V: track 116.1 -> 114.1 mm
- net 1.1V: track 1.97 -> 0.00 mm
- net Net-(U20-IN): track 1.62 -> 0.00 mm
- net /SIP B: ADC + Crystals/USB_VBUS: track 63.6 -> 64.1 mm
- net GND: vias 807 -> 809
- added copper zone on F.Cu, net 1.1V
