File: oresat-live-card/oresat-live-card.kicad_sch (KiCad schematic)
At the start: 17 parts, among them J1 SM14B-SHLS-TF, J10 SM06B-SRSS-TB, J12 U.FL, J2 SM06B-SRSS-TB, J4 TFM-120-01-L-D-RA, J6 SMPM, J8 SMPM, J9 U.FL

Commit message: BOM changes
Updated components outside of RF path to on hand parts.
Parts:
- J1: value SM14B-SHLS-TF -> TFM-120-01-L-D-RA; footprint oresat-connectors:J-JST-SM14BSHLSTF -> oresat-connectors:J-SAMTEC-TFM-120-X1-XXX-D-RA; DPN 455-SM14B-SHLS-TFCT-ND -> SAM10145-ND; MFR JST -> Samtec Inc.; MPN SM14B-SHLS-TF -> TFM-120-01-L-D-RA
- J10, J2: value SM06B-SRSS-TB -> GRPB041VWVN-RC; footprint oresat-live-card:CONN_SM06B-SRSS-TB_JST -> Connector_PinHeader_1.27mm:PinHeader_1x04_P1.27mm_Vertical; DPN 455-SM06B-SRSS-TBCT-ND -> S9014E-04-ND; MFR JST Commercial -> Sulins Connector Solutions; MPN SM06B-SRSS-TB -> GRPB041VWVN-RC
- J12, J9: value U.FL -> Conn_01x02; footprint Connector_Coaxial:U.FL_Molex_MCRF_73412-0110_Vertical -> Connector_PinHeader_2.54mm:PinHeader_1x02_P2.54mm_Vertical; DIS DigiKey -> (none); DPN H11891CT-ND -> (none); MFR Hirose Electric Co Ltd -> (none); MPN U.FL-R-SMT-1(10) -> (none)
- J4: value TFM-120-01-L-D-RA -> SMPM; footprint oresat-connectors:J-SAMTEC-TFM-120-X1-XXX-D-RA -> oresat-connectors:J-MOLEX-SMPM-073300-002X; DPN SAM10145-ND -> WM10772-ND; MFR Samtec Inc. -> MOLEX; MPN TFM-120-01-L-D-RA -> 0733000020
- J6, J8: value SMPM -> U.FL; footprint oresat-connectors:J-MOLEX-SMPM-073300-002X -> Connector_Coaxial:U.FL_Molex_MCRF_73412-0110_Vertical; DPN WM10772-ND -> H11891CT-ND; MFR MOLEX -> Hirose Electric Co Ltd; MPN 0733000020 -> U.FL-R-SMT-1(10)
- PCB1: value ORESAT-CARD-V1.3-GENERIC-1RF-POS1 -> MMBT2907; footprint oresat-pcbs:ORESAT-CARD-V1.3-2RF-LEFT -> Package_TO_SOT_SMD:SOT-23; DIS N/A -> DigiKey; DPN N/A -> 1727-1884-1-ND; MFR N/A -> Nexperia; MPN N/A -> PMBT2907A,235
- PCBA1: value WF-NP9202WF -> DMN2050LQ-7; footprint oresat-live-card:WF-NP9202 -> Package_TO_SOT_SMD:SOT-23; DIS N/A -> DigiKey; DPN N/A -> 31-DMN2050LQ-7CT-ND; MFR Unknown -> Diodes Incorporated; MPN Unknown -> DMN2050LQ-7
- TP159: value 0.03x0.04 -> THGBMJG8C4LBAU8; footprint oresat-misc:TestPoint-0.75mm-th -> oresat-ics:BGA-153(11.5X13)(EMMC-BA); DIS (none) -> Mouser; DPN (none) -> 757-THGBMJG8C4LBAU8; MFR (none) -> Kioxia; MPN (none) -> THGBMJG8C4LBAU8

Commit message: Very minor layout changes
Connections:
- net WiFi LNA/RF_DET_IN renamed WiFi LNA/AR9271_IN
Other:
- sheet WiFi LNA ports: added AR9271_IN; removed RF_DET_IN
Changed lines of the file:
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@@
 			)
 		)
-		(pin "RF_DET_IN" input
+		(pin "AR9271_IN" input
 			(at 407.67 190.5 0)
 			(effects
