File: oresat-live-card/oresat-live-card-sch-sip-b.kicad_sch (KiCad schematic)
At the start: 25 parts, among them U23 RCLAMP0504FB, U7 OSD3358-512M-BSM, Y1 24MHz, Y2 32.768KHZ

Commit message: Organizational changes
Updated hierarchical labels and other misc schematic fixes
Parts:
- removed R100: 0, oresat-passives:0603-C-NOSILK, symbol Device:R_Small_US
Changed lines of the file:
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@@
-	)
-	(junction
-		(at 259.08 167.64)
-		(diameter 0)
-		(color 0 0 0 0)
 	)
 	(junction
@@
 	(wire
 		(pts
-			(xy 266.7 163.83) (xy 269.24 163.83)
-		)
-		(stroke
-			(width 0)
-			(type default)
-		)
-	)
-	(wire
-		(pts
 			(xy 243.84 157.48) (xy 247.65 157.48)
 		)
@@
 	(wire
 		(pts
-			(xy 259.08 163.83) (xy 261.62 163.83)
-		)
-		(stroke
-			(width 0)
-			(type default)
-		)
-	)
-	(wire
-		(pts
 			(xy 243.84 78.74) (xy 248.92 78.74)
 		)
@@
 	(wire
 		(pts
-			(xy 259.08 163.83) (xy 259.08 167.64)
-		)
-		(stroke
-			(width 0)
-			(type default)
-		)
-	)
-	(wire
-		(pts
 			(xy 107.95 149.86) (xy 125.73 149.86)
 		)
@@
 	(wire
 		(pts
-			(xy 259.08 167.64) (xy 264.16 167.64)
-		)
-		(stroke
-			(width 0)
-			(type default)
-		)
-	)
-	(wire
-		(pts
 			(xy 182.88 81.28) (xy 152.4 81.28)
 		)
@@
 	(wire
 		(pts
-			(xy 243.84 167.64) (xy 259.08 167.64)
+			(xy 243.84 167.64) (xy 264.16 167.64)
 		)
 		(stroke
@@
 	)
 	(symbol
-		(lib_id "Device:R_Small_US")
-		(at 264.16 163.83 270)
-		(unit 1)
-		(body_style 1)
-		(exclude_from_sim no)
-		(in_bom yes)
-		(on_board yes)
-		(in_pos_files yes)
-		(dnp no)
-		(property "Reference" "R100"
-			(at 266.954 157.099 90)
-			(show_name no)
-			(do_not_autoplace no)
-			(effects
-				(font
-					(size 1.778 1.5113)
-				)
-				(justify right top)
-			)
-		)
-		(property "Value" "0"
-			(at 262.636 161.544 90)
-			(show_name no)
-			(do_not_autoplace no)
-			(effects
-				(font
-					(size 1.778 1.5113)
-				)
-				(justify right bottom)
-			)
-		)
-		(property "Footprint" "oresat-passives:0603-C-NOSILK"
-			(at 264.16 163.83 0)
-			(hide yes)
-			(show_name no)
-			(do_not_autoplace no)
-			(effects
-				(font
-					(size 1.27 1.27)
-				)
-			)
-		)
-		(property "Datasheet" ""
-			(at 264.16 163.83 0)
-			(hide yes)
-			(show_name no)
-			(do_not_autoplace no)
-			(effects
-				(font
-					(size 1.27 1.27)
-				)
-			)
-		)
-		(property "Description" "Resistor, small US symbol"
-			(at 264.16 163.83 0)
-			(hide yes)
-			(show_name no)
-			(do_not_autoplace no)
-			(effects
-				(font
-					(size 1.27 1.27)
-				)
-			)
-		)
-		(property "MPN" "ERJ-3GEY0R00V"
-			(at 264.16 163.83 0)
-			(hide yes)
-			(show_name no)
-			(do_not_autoplace no)
-			(effects
-				(font
-					(size 1.27 1.27)
-				)
-			)
-		)
-		(property "DPN" "P0.0GCT-ND "
-			(at 264.16 163.83 0)
-			(hide yes)
-			(show_name no)
-			(do_not_autoplace no)
-			(effects
-				(font
-					(size 1.27 1.27)
-				)
-			)
-		)
-		(property "MFR" "Panasonic "
-			(at 264.16 163.83 0)
-			(hide yes)
-			(show_name no)
-			(do_not_autoplace no)
-			(effects
-				(font
-					(size 1.27 1.27)
-				)
-			)
-		)
-		(property "DIS" "DigiKey"
-			(at 264.16 163.83 0)
-			(hide yes)
-			(show_name no)
-			(do_not_autoplace no)
-			(effects
-				(font
-					(size 1.27 1.27)
-				)
-			)
-		)
-		(pin "1"
-		)
-		(pin "2"
-		)
-		(instances
-			(project "oresat-live-card"
-				(path "/748bdd2d-da0a-4240-ba60-0bf881d2ec56/49f5f571-d1f9-4350-855b-6ca6690b0a90"
-					(reference "R100")
-					(unit 1)
-				)
-			)
-		)
-	)
-	(symbol
 		(lib_id "Device:C_Small")
 		(at 134.62 111.76 270)
@@
 					(unit 1)
 				)
-			)
-		)
-	)
-	(symbol
-		(lib_id "power:+5V")
-		(at 269.24 163.83 0)
-		(unit 1)
-		(body_style 1)
-		(exclude_from_sim no)
-		(in_bom yes)
-		(on_board yes)
-		(in_pos_files yes)
-		(dnp no)
-		(property "Reference" "#PWR0172"
-			(at 269.24 167.64 0)
-			(hide yes)
-			(show_name no)
-			(do_not_autoplace no)
-			(effects
-				(font
-					(size 1.27 1.27)
-				)
-			)
-		)
-		(property "Value" "+5V"
-			(at 269.24 160.274 0)
-			(show_name no)
-			(do_not_autoplace no)
-			(effects
-				(font
-					(size 1.27 1.27)
-				)
-			)
-		)
-		(property "Footprint" ""
-			(at 269.24 163.83 0)
-			(hide yes)
-			(show_name no)
-			(do_not_autoplace no)
-			(effects
-				(font
-					(size 1.27 1.27)
-				)
-			)
-		)
-		(property "Datasheet" ""
-			(at 269.24 163.83 0)
-			(hide yes)
-			(show_name no)
-			(do_not_autoplace no)
-			(effects
-				(font
-					(size 1.27 1.27)
-				)
-			)
-		)
-		(property "Description" "Power symbol creates a global label with name \"+5V\""
-			(at 269.24 163.83 0)
-			(hide yes)
-			(show_name no)
-			(do_not_autoplace no)
-			(effects
-				(font
-					(size 1.27 1.27)
-				)
-			)
-		)
-		(pin "1"
-		)
-		(instances
-			(project "oresat-live-card"
-				(path "/748bdd2d-da0a-4240-ba60-0bf881d2ec56/49f5f571-d1f9-4350-855b-6ca6690b0a90"
-					(reference "#PWR0172")
-					(unit 1)
-				)

Commit message: Schematic and PCB update
updated hierarchy labels to have more clarifying names. Fixed RF connector symbol to footprint issues. Linked footprints and 3d models. Added DRC error clearance to ignore of specific RF class. Fixed most of all the DRC warnings and errors outside emmc and silkscreen on exposed copper
Connections:
- net RX_DET_OUT renamed RF/RX_IN_DETECTED
Changed lines of the file:
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@@
 		)
 	)
-	(hierarchical_label "RX_DET_OUT"
+	(hierarchical_label "RF{slash}RX_IN_DETECTED"
 		(shape input)
 		(at 259.08 142.24 0)

Commit message: BOM changes
Updated components outside of RF path to on hand parts.
Parts:
- C19, C22, C23, C25, C26, C29, C30: footprint oresat-passives:0603-C-NOSILK -> oresat-passives:0603-C
- FB2: value BLM18KG300TH1D -> QPQ1907SR; footprint oresat-live-card:0603 -> oresat-ics:QPQ1907SR; DPN 490-13263-1-ND -> 2312-QPQ1907SRCT-ND; MFR Murata Electronics -> Qorvo; MPN BLM18KG300JH1D -> QPQ1907SR
- R13: value 1M -> 100k; footprint oresat-passives:0603-C-NOSILK -> oresat-live-card:ARRAY_EXBA-M; DPN P1.00MHCT-ND -> U7104CT-ND; MPN ERJ-3EKF1004V -> EXB-A10P104J
- R18: value 10k -> 100k; DPN P10.0KHCT-ND -> RMCF0603FT100KCT-ND; MFR Panasonic -> Stackpole Electronics; MPN ERJ-3EKF1002V -> RMCF0603FT100K
- R96: value 0 -> 9.53k; footprint oresat-passives:0603-C-NOSILK -> oresat-passives:0603-C; DPN P0.0GCT-ND -> P9.53KHCT-ND; MPN ERJ-3GEY0R00V -> ERJ-3EKF9531V
- TP10, TP12, TP144, TP29, TP5, TP6, TP7, TP8: footprint oresat-misc:TestPoint_Pad_D1.0mm -> oresat-misc:TestPoint-0.75mm-th
- U23: value RCLAMP0504FB -> SN74LVC1G32QDBVRQ1; footprint oresat-live-card:SC70-6 -> Package_TO_SOT_SMD:SOT-23-5; DPN RCLAMP0504FBTCTCT-ND -> 296-24202-1-ND; MFR Semtech Corporation -> Texas Instruments; MPN RCLAMP0504FBTCT -> SN74LVC1G32QDBVRQ1
- U7: value OSD3358-512M-BSM -> TPS2041BQDBVRQ1; footprint oresat-ics:U-Octavo-OSD335X-BGA-256 -> oresat-live-card:DBV5; DPN 1676-1002-ND -> 296-25159-1-ND; MFR Octavo Systems -> Texas Instruments; MPN OSD3358-512M-BSM -> TPS2041BQDBVRQ1
Changed lines of the file:
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@@
 			)
 		)
-		(property "Footprint" "oresat-misc:TestPoint_Pad_D1.0mm"
+		(property "Footprint" "oresat-misc:TestPoint-0.75mm-th"
 			(at 170.18 175.26 0)
 			(hide yes)
@@
 			)
 		)
-		(property "Value" "10k"
+		(property "Value" "100k"
 			(at 282.194 123.444 0)
 			(show_name no)
@@
 			)
 		)
-		(property "Datasheet" ""
+		(property "Datasheet" "https://www.seielect.com/catalog/SEI-RMCF_RMCP.pdf"
 			(at 288.29 123.19 0)
 			(hide yes)
@@
 			)
 		)
-		(property "Description" "Resistor, small US symbol"
+		(property "Description" "100 kOhms ±1% 0.1W, 1/10W Chip Resistor 0603 (1608 Metric) Automotive AEC-Q200 Thick Film"
 			(at 288.29 123.19 0)
 			(hide yes)
@@
 			)
 		)
-		(property "MPN" "ERJ-3EKF1002V"
+		(property "MPN" "RMCF0603FT100K"
 			(at 288.29 123.19 0)
 			(hide yes)
@@
 			)
 		)
-		(property "DPN" "P10.0KHCT-ND "
+		(property "DPN" "RMCF0603FT100KCT-ND"
 			(at 288.29 123.19 0)
 			(hide yes)
@@
 			)
 		)
-		(property "MFR" "Panasonic "
+		(property "MFR" "Stackpole Electronics"
 			(at 288.29 123.19 0)
 			(hide yes)
@@
 			)
 		)
-		(property "Footprint" "oresat-misc:TestPoint_Pad_D1.0mm"
+		(property "Footprint" "oresat-misc:TestPoint-0.75mm-th"
 			(at 238.76 129.54 0)
 			(hide yes)
@@
 			)
 		)
-		(property "Footprint" "oresat-passives:0603-C-NOSILK"
+		(property "Footprint" "oresat-passives:0603-C"
 			(at 288.29 133.35 0)
 			(hide yes)
@@
 			)
 		)
-		(property "Footprint" "oresat-passives:0603-C-NOSILK"
+		(property "Footprint" "oresat-passives:0603-C"
 			(at 248.92 92.71 0)
 			(hide yes)
@@
 			)
 		)
-		(property "Value" "1M"
+		(property "Value" "100k"
 			(at 157.48 91.44 0)
 			(show_name no)
@@
 			)
 		)
-		(property "Footprint" "oresat-passives:0603-C-NOSILK"
+		(property "Footprint" "oresat-live-card:ARRAY_EXBA-M"
 			(at 152.4 88.9 0)
 			(hide yes)
@@
 			)
 		)
-		(property "Description" "Resistor, small US symbol"
+		(property "Description" "RES ARRAY 8 RES 100K OHM 2512"
 			(at 152.4 88.9 0)
 			(hide yes)
@@
 			)
 		)
-		(property "MPN" "ERJ-3EKF1004V"
+		(property "MPN" "EXB-A10P104J"
 			(at 152.4 88.9 0)
 			(hide yes)
@@
 			)
 		)
-		(property "DPN" "P1.00MHCT-ND "
+		(property "DPN" "U7104CT-ND "
 			(at 152.4 88.9 0)
 			(hide yes)
@@
 			)
 		)
-		(property "Footprint" "oresat-misc:TestPoint_Pad_D1.0mm"
+		(property "Footprint" "oresat-misc:TestPoint-0.75mm-th"
 			(at 245.11 167.64 0)
 			(hide yes)
@@
 			)
 		)
-		(property "Footprint" "oresat-passives:0603-C-NOSILK"
+		(property "Footprint" "oresat-passives:0603-C"
 			(at 134.62 111.76 0)
 			(hide yes)
@@
 			)
 		)
-		(property "Footprint" "oresat-passives:0603-C-NOSILK"
+		(property "Footprint" "oresat-passives:0603-C"
 			(at 134.62 127 0)
 			(hide yes)
@@
 			)
 		)
-		(property "Footprint" "oresat-misc:TestPoint_Pad_D1.0mm"
+		(property "Footprint" "oresat-misc:TestPoint-0.75mm-th"
 			(at 247.65 170.18 0)
 			(hide yes)
@@
 			)
 		)
-		(property "Footprint" "oresat-misc:TestPoint_Pad_D1.0mm"
+		(property "Footprint" "oresat-misc:TestPoint-0.75mm-th"
 			(at 237.49 157.48 0)
 			(hide yes)
@@
 			)
 		)
-		(property "Footprint" "oresat-passives:0603-C-NOSILK"
+		(property "Footprint" "oresat-passives:0603-C"
 			(at 127 81.28 0)
 			(hide yes)
@@
 			)
 		)
-		(property "Value" "OSD3358-512M-BSM"
+		(property "Value" "TPS2041BQDBVRQ1"
 			(at 187.96 66.04 0)
 			(show_name no)
@@
 			)
 		)
-		(property "Footprint" "oresat-ics:U-Octavo-OSD335X-BGA-256"
+		(property "Footprint" "oresat-live-card:DBV5"
 			(at 213.36 16.51 0)
 			(hide yes)
@@
 			)
 		)
-		(property "Datasheet" ""
+		(property "Datasheet" "https://www.ti.com/lit/ds/symlink/tps2041b-q1.pdf?HQS=dis-dk-null-digikeymode-dsf-pf-null-wwe&ts=1651525711603&ref_url=https%253A%252F%252Fwww.ti.com%252Fgeneral%252Fdocs%252Fsuppproductinfo.tsp%253FdistId%253D10%2526gotoUrl%253Dhttps%253A%252F%252Fwww.ti.com%252Flit%252Fgpn%252Ftps2041b-q1"
 			(at 213.36 124.46 0)
 			(hide yes)
@@
 			)
 		)
-		(property "Description" "OSD335x Embedded Module 1GHz 512MB"
+		(property "Description" "Power Switch/Driver 1:1 N-Channel 500mA"
 			(at 213.36 124.46 0)
 			(hide yes)
@@
 			)
 		)
-		(property "MPN" "OSD3358-512M-BSM"
+		(property "MPN" "TPS2041BQDBVRQ1"
 			(at 213.36 124.46 0)
 			(hide yes)
@@
 			)
 		)
-		(property "DPN" "1676-1002-ND "
+		(property "DPN" "296-25159-1-ND "
 			(at 213.36 124.46 0)
 			(hide yes)
@@
 			)
 		)
-		(property "MFR" "Octavo Systems "
+		(property "MFR" "Texas Instruments "
 			(at 213.36 124.46 0)
 			(hide yes)
@@
 			)
 		)
-		(property "Footprint" "oresat-misc:TestPoint_Pad_D1.0mm"
+		(property "Footprint" "oresat-misc:TestPoint-0.75mm-th"
 			(at 237.49 149.86 0)
 			(hide yes)
@@
 			)
 		)
-		(property "Value" "BLM18KG300TH1D"
+		(property "Value" "QPQ1907SR"
 			(at 118.11 167.64 0)
 			(hide yes)
@@
 			)
 		)
-		(property "Footprint" "oresat-live-card:0603"
+		(property "Footprint" "oresat-ics:QPQ1907SR"
 			(at 118.11 167.64 0)
 			(hide yes)
@@
 			)
 		)
-		(property "Datasheet" ""
+		(property "Datasheet" "https://www.qorvo.com/products/d/da006450"
 			(at 118.11 167.64 0)
 			(hide yes)
@@
 			)
 		)
-		(property "Description" "FERRITE BEAD 30 OHM 0603 1 LN"
+		(property "Description" "2.4GHZ WI-FI LTE COEXBOOST BAW F"
 			(at 118.11 167.64 0)
 			(hide yes)
@@
 			)
 		)
-		(property "MPN" "BLM18KG300JH1D"
+		(property "MPN" "QPQ1907SR"
 			(at 118.11 167.64 0)
 			(hide yes)
@@
 			)
 		)
-		(property "DPN" "490-13263-1-ND "
+		(property "DPN" "2312-QPQ1907SRCT-ND"
 			(at 118.11 167.64 90)
 			(hide yes)
@@
 			)
 		)
-		(property "MFR" "Murata Electronics "
+		(property "MFR" "Qorvo"
 			(at 118.11 167.64 90)
 			(hide yes)
@@
 			)
 		)
-		(property "Footprint" "oresat-misc:TestPoint_Pad_D1.0mm"
+		(property "Footprint" "oresat-misc:TestPoint-0.75mm-th"
 			(at 170.18 177.8 0)
 			(hide yes)
@@
 			)
 		)
-		(property "Footprint" "oresat-misc:TestPoint_Pad_D1.0mm"
+		(property "Footprint" "oresat-misc:TestPoint-0.75mm-th"
 			(at 170.18 180.34 0)
 			(hide yes)
@@
 			)
 		)
-		(property "Value" "RCLAMP0504FB"
+		(property "Value" "SN74LVC1G32QDBVRQ1"
 			(at 99.06 182.88 0)
 			(show_name no)
@@
 			)
 		)
-		(property "Footprint" "oresat-live-card:SC70-6"
+		(property "Footprint" "Package_TO_SOT_SMD:SOT-23-5"
 			(at 113.03 193.04 0)
 			(hide yes)
@@
 			)
 		)
-		(property "Datasheet" ""
+		(property "Datasheet" "-- mixed values --"
 			(at 113.03 193.04 0)
 			(hide yes)
@@
 			)
 		)
-		(property "Description" "TVS DIODE 5V 17.5V SC70-6"
+		(property "Description" "-- mixed values --"
 			(at 113.03 193.04 0)
 			(hide yes)
@@
 			)
 		)
-		(property "MPN" "RCLAMP0504FBTCT"
+		(property "MPN" "SN74LVC1G32QDBVRQ1"
 			(at 113.03 193.04 0)
 			(hide yes)
@@
 			)
 		)
-		(property "DPN" "RCLAMP0504FBTCTCT-ND "
+		(property "DPN" "296-24202-1-ND"
 			(at 113.03 193.04 0)
 			(hide yes)
@@
 			)
 		)
-		(property "MFR" "Semtech Corporation "
+		(property "MFR" "Texas Instruments"
 			(at 113.03 193.04 0)
 			(hide yes)
@@
 			)
 		)
-		(property "Footprint" "oresat-passives:0603-C-NOSILK"
+		(property "Footprint" "oresat-passives:0603-C"
 			(at 124.46 182.88 0)
 			(hide yes)
@@
 			)
 		)
-		(property "Value" "0"
+		(property "Value" "9.53k"
 			(at 253.746 185.674 0)
 			(show_name no)
@@
 			)
 		)
-		(property "Footprint" "oresat-passives:0603-C-NOSILK"
+		(property "Footprint" "oresat-passives:0603-C"
 			(at 259.08 180.34 0)
 			(hide yes)
@@
 			)
 		)
-		(property "Description" "Resistor, small US symbol"
+		(property "Description" "RES 9.53K OHM 1% 1/10W 0603"
 			(at 259.08 180.34 0)
 			(hide yes)
@@
 			)
 		)
-		(property "MPN" "ERJ-3GEY0R00V"
+		(property "MPN" "ERJ-3EKF9531V "
 			(at 259.08 180.34 0)
 			(hide yes)
@@
 			)
 		)
-		(property "DPN" "P0.0GCT-ND "
+		(property "DPN" "P9.53KHCT-ND "
 			(at 259.08 180.34 0)
 			(hide yes)
@@
 			)
 		)
-		(property "Footprint" "oresat-passives:0603-C-NOSILK"
+		(property "Footprint" "oresat-passives:0603-C"
 			(at 127 96.52 0)
 			(hide yes)

Commit message: Cleanup of main sheet, no changes to functionality
Other:
- moved on the sheet: C19, C22, C23, C25, C26, C29, C30, FB2, R13, R18, R27, R96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

Commit message: BOM changed to match older version
Parts:
- C19, C22, C29, C30: footprint oresat-passives:0603-C -> oresat-passives:0603-C-NOSILK; DPN 445-5629-1-ND -> 445-5629-1-ND; MFR TDK Corporation -> TDK Corporation; MPN CGA3E2C0G1H120J080AA -> CGA3E2C0G1H120J080AA
- C23, C25, C26: footprint oresat-passives:0603-C -> oresat-passives:0603-C-NOSILK; DPN 445-5667-1-ND -> 445-5667-1-ND; MFR TDK Corporation -> TDK Corporation; MPN CGA3E2X7R1E104K080AA -> CGA3E2X7R1E104K080AA
- FB2: value QPQ1907SR -> BLM18KG300TH1D; footprint oresat-ics:QPQ1907SR -> oresat-live-card:0603; DPN 2312-QPQ1907SRCT-ND -> 490-13263-1-ND; MFR Qorvo -> Murata Electronics; MPN QPQ1907SR -> BLM18KG300JH1D
- R13: value 100k -> 1M; footprint oresat-live-card:ARRAY_EXBA-M -> oresat-passives:0603-C-NOSILK; DPN U7104CT-ND -> P1.00MHCT-ND; MFR Panasonic -> Panasonic; MPN EXB-A10P104J -> ERJ-3EKF1004V
- R18: value 100k -> 10k; MFR Stackpole Electronics -> Panasonic
- R96: value 9.53k -> 0; footprint oresat-passives:0603-C -> oresat-passives:0603-C-NOSILK; DPN P9.53KHCT-ND -> P0.0GCT-ND; MFR Panasonic -> Panasonic; MPN ERJ-3EKF9531V -> ERJ-3GEY0R00V
- TP10, TP12, TP144, TP29, TP5, TP6, TP7, TP8: footprint oresat-misc:TestPoint-0.75mm-th -> oresat-misc:TestPoint_Pad_D1.0mm
- U23: value SN74LVC1G32QDBVRQ1 -> RCLAMP0504FB; footprint Package_TO_SOT_SMD:SOT-23-5 -> oresat-live-card:SC70-6; DPN 296-24202-1-ND -> RCLAMP0504FBTCTCT-ND; MFR Texas Instruments -> Semtech Corporation; MPN SN74LVC1G32QDBVRQ1 -> RCLAMP0504FBTCT
- U7: value TPS2041BQDBVRQ1 -> OSD3358-512M-BSM; footprint oresat-live-card:DBV5 -> oresat-ics:U-Octavo-OSD335X-BGA-256; DPN 296-25159-1-ND -> 1676-1002-ND; MFR Texas Instruments -> Octavo Systems; MPN TPS2041BQDBVRQ1 -> OSD3358-512M-BSM
- Y1: DPN XC2580CT-ND -> XC2580CT-ND; MFR ECS Inc. -> ECS Inc.
- Y2: DPN 535-9542-1-ND -> 535-9542-1-ND; MFR Abracon LLC -> Abracon LLC
