File: oresat-live-card/oresat-live-card-sch-sip-b.kicad_sch (KiCad schematic)
At the start: 24 parts, among them U23 RCLAMP0504FB, U7 OSD3358-512M-BSM, Y1 24MHz, Y2 32.768KHZ

Commit message: mostly just polish after BOM fixes
Parts:
- TP10, TP12, TP144, TP29, TP5, TP6, TP7, TP8: now left out of the parts list
Connections:
- net OSC0_IN: now also Y1.3; no longer Y1.1
- net OSC0_OUT: now also Y1.1; no longer Y1.3
Other:
- note added: "All resistors 0603 +/- 1% unless marked and AEQ certified unless otherwise marked. All caps are 0603 10% X5R or better and Vw >= 25 V and AEQ certified unless otherwise marked."
- note removed: "All caps are 0603 ceramic 10% X7R Vw>=16V unless marked"
- note removed: "All resistors 0603 +/- 1% unless marked"
Changed lines of the file:
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@@
 	(text "VIN_USB can power the OSD335x"
 		(exclude_from_sim no)
-		(at 157.48 147.32 0)
+		(at 115.062 147.32 0)
 		(effects
 			(font
-				(size 1.778 1.5113)
-			)
-			(justify left bottom)
-		)
-	)
-	(text "All caps are 0603 ceramic 10% X7R Vw>=16V unless marked"
-		(exclude_from_sim no)
-		(at 126.238 264.922 0)
-		(effects
-			(font
-				(size 1.778 1.5113)
+				(size 1.27 1.27)
 			)
 			(justify left bottom)
 		)
 	)
-	(text "All resistors 0603 +/- 1% unless marked"
+	(text "All resistors 0603 +/- 1% unless marked and AEQ certified unless otherwise marked.\nAll caps are 0603 10% X5R or better and Vw >= 25 V and AEQ certified unless otherwise marked."
 		(exclude_from_sim no)
-		(at 126.238 262.382 0)
+		(at 112.776 265.938 0)
 		(effects
 			(font
@@
 		(body_style 1)
 		(exclude_from_sim no)
-		(in_bom yes)
+		(in_bom no)
 		(on_board yes)
 		(in_pos_files yes)
@@
 			(effects
 				(font
-					(size 1.778 1.778)
+					(size 1.27 1.27)
 				)
 				(justify left bottom)
@@
 			(effects
 				(font
-					(size 1.778 1.5113)
+					(size 1.27 1.27)
 				)
 				(justify left bottom)
@@
 			(effects
 				(font
-					(size 1.778 1.5113)
+					(size 1.27 1.27)
 				)
 				(justify left bottom)
@@
 		(lib_id "Device:Crystal_GND24")
 		(at 166.37 88.9 270)
+		(mirror x)
 		(unit 1)
 		(body_style 1)
@@
 		(dnp no)
 		(property "Reference" "Y1"
-			(at 166.37 74.93 90)
+			(at 166.37 102.87 90)
 			(show_name no)
 			(do_not_autoplace no)
 			(effects
 				(font
-					(size 1.778 1.778)
+					(size 1.27 1.27)
 				)
 				(justify bottom)
@@
 		)
 		(property "Value" "24MHz"
-			(at 166.37 76.2 90)
+			(at 166.37 101.6 90)
 			(show_name no)
 			(do_not_autoplace no)
 			(effects
 				(font
-					(size 1.778 1.778)
+					(size 1.27 1.27)
 				)
 				(justify top)
@@
 		(body_style 1)
 		(exclude_from_sim no)
-		(in_bom yes)
+		(in_bom no)
 		(on_board yes)
 		(in_pos_files yes)
@@
 			(effects
 				(font
-					(size 1.778 1.778)
+					(size 1.27 1.27)
 				)
 				(justify right top)
@@
 			(effects
 				(font
-					(size 1.778 1.5113)
+					(size 1.27 1.27)
 				)
 				(justify left bottom)
@@
 			(effects
 				(font
-					(size 1.778 1.5113)
+					(size 1.27 1.27)
 				)
 				(justify left bottom)
@@
 			(effects
 				(font
-					(size 1.778 1.5113)
+					(size 1.27 1.27)
 				)
 				(justify left bottom)
@@
 			(effects
 				(font
-					(size 1.778 1.5113)
+					(size 1.27 1.27)
 				)
 				(justify left bottom)
@@
 			(effects
 				(font
-					(size 1.778 1.5113)
+					(size 1.27 1.27)
 				)
 				(justify left bottom)
@@
 			(effects
 				(font
-					(size 1.778 1.5113)
+					(size 1.27 1.27)
 				)
 				(justify left top)
@@
 		(body_style 1)
 		(exclude_from_sim no)
-		(in_bom yes)
+		(in_bom no)
 		(on_board yes)
 		(in_pos_files yes)
@@
 			(effects
 				(font
-					(size 1.778 1.778)
+					(size 1.27 1.27)
 				)
 				(justify left bottom)
@@
 			(effects
 				(font
-					(size 1.778 1.5113)
+					(size 1.27 1.27)
 				)
 				(justify left bottom)
@@
 			(effects
 				(font
-					(size 1.778 1.5113)
+					(size 1.27 1.27)
 				)
 				(justify left bottom)
@@
 			(effects
 				(font
-					(size 1.778 1.5113)
+					(size 1.27 1.27)
 				)
 				(justify left bottom)
@@
 			(effects
 				(font
-					(size 1.778 1.5113)
+					(size 1.27 1.27)
 				)
 				(justify left bottom)
@@
 			(effects
 				(font
-					(size 1.27 1.0795)
+					(size 1.27 1.27)
 				)
 				(justify right top)
@@
 			(effects
 				(font
-					(size 1.27 1.0795)
+					(size 1.27 1.27)
 				)
 				(justify right top)
@@
 		(body_style 1)
 		(exclude_from_sim no)
-		(in_bom yes)
+		(in_bom no)
 		(on_board yes)
 		(in_pos_files yes)
@@
 			(effects
 				(font
-					(size 1.778 1.778)
+					(size 1.27 1.27)
 				)
 				(justify left bottom)
@@
 		(body_style 1)
 		(exclude_from_sim no)
-		(in_bom yes)
+		(in_bom no)
 		(on_board yes)
 		(in_pos_files yes)
@@
 			(effects
 				(font
-					(size 1.778 1.778)
+					(size 1.27 1.27)
 				)
 				(justify right top)
@@
 			(effects
 				(font
-					(size 1.778 1.5113)
+					(size 1.27 1.27)
 				)
 				(justify right top)
@@
 			(effects
 				(font
-					(size 1.778 1.5113)
+					(size 1.27 1.27)
 				)
 				(justify right top)
@@
 			(effects
 				(font
-					(size 1.778 1.5113)
+					(size 1.27 1.27)
 				)
 				(justify left top)
@@
 			(effects
 				(font
-					(size 1.778 1.5113)
+					(size 1.27 1.27)
 				)
 				(justify left bottom)
@@
 		(body_style 1)
 		(exclude_from_sim no)
-		(in_bom yes)
+		(in_bom no)
 		(on_board yes)
 		(in_pos_files yes)
@@
 			(effects
 				(font
-					(size 1.778 1.778)
+					(size 1.27 1.27)
 				)
 				(justify right top)
@@
 			(effects
 				(font
-					(size 1.778 1.778)
+					(size 1.27 1.27)
 				)
 				(justify right top)
@@
 		(body_style 1)
 		(exclude_from_sim no)
-		(in_bom yes)
+		(in_bom no)
 		(on_board yes)
 		(in_pos_files yes)
@@
 			(effects
 				(font
-					(size 1.778 1.778)
+					(size 1.27 1.27)
 				)
 				(justify left bottom)
@@
 		(body_style 1)
 		(exclude_from_sim no)
-		(in_bom yes)
+		(in_bom no)
 		(on_board yes)
 		(in_pos_files yes)
@@
 			(effects
 				(font
-					(size 1.778 1.778)
+					(size 1.27 1.27)
 				)
 				(justify left bottom)
@@
 			(effects
 				(font
-					(size 1.27 1.0795)
+					(size 1.27 1.27)
 				)
 				(justify left bottom)
@@
 			(effects
 				(font
-					(size 1.27 1.0795)
+					(size 1.27 1.27)
 				)
 				(justify left bottom)
@@
 			)
 		)
-		(property "Datasheet" "-- mixed values --"
+		(property "Datasheet" ""
 			(at 142.24 193.04 0)
 			(hide yes)
@@
 			(effects
 				(font
-					(size 1.778 1.5113)
+					(size 1.27 1.27)
 				)
 				(justify left bottom)
@@
 			(effects
 				(font
-					(size 1.778 1.5113)
+					(size 1.27 1.27)
 				)
 				(justify left bottom)
@@
 			(effects
 				(font
-					(size 1.778 1.5113)
+					(size 1.27 1.27)
 				)
 				(justify right top)
@@
 			(effects
 				(font
-					(size 1.778 1.5113)
+					(size 1.27 1.27)
 				)
 				(justify right bottom)
@@
 			(effects
 				(font
-					(size 1.778 1.5113)
+					(size 1.27 1.27)
 				)
 				(justify right top)
@@
 			(effects
 				(font
-					(size 1.778 1.5113)
+					(size 1.27 1.27)
 				)
 				(justify right top)
@@
 			(effects
 				(font
-					(size 1.778 1.5113)
+					(size 1.27 1.27)
 				)
 				(justify left top)
@@
 			(effects
 				(font
-					(size 1.778 1.5113)
+					(size 1.27 1.27)
 				)
 				(justify left top)

Commit message: Updated BOM
Parts:
- C19, C22, C29, C30: DPN 445-5629-1-ND -> 478-KAM15ACG2A120KTTR-ND; MFR TDK Corporation -> KYOCERA AVX; MPN CGA3E2C0G1H120J080AA -> KAM15ACG2A120KT
- C23, C25, C26: value 100n -> 0.1u; DPN 445-5667-1-ND -> 399-6856-1-ND; MFR TDK Corporation -> KEMET; MPN CGA3E2X7R1E104K080AA -> C0603C104K5RACAUTO
- R13: DPN P1.00MHCT-ND -> RMCF0603FT1M00CT-ND; MFR Panasonic -> Stackpole Electronics; MPN ERJ-3EKF1004V -> RMCF0603FT1M00
- R18: DPN RMCF0603FT100KCT-ND -> RMCF0603FT10K0CT-ND; MFR Panasonic -> Stackpole Electronics; MPN RMCF0603FT100K -> RMCF0603FT10K0
- R96: DPN P0.0GCT-ND -> RMCF0603ZT0R00CT-ND; MFR Panasonic -> Stackpole Electronics; MPN ERJ-3GEY0R00V -> RMCF0603ZT0R00
Changed lines of the file:
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@@
 			)
 		)
-		(property "Description" "100 kOhms ±1% 0.1W, 1/10W Chip Resistor 0603 (1608 Metric) Automotive AEC-Q200 Thick Film"
+		(property "Description" "10 kOhms ±1% 0.1W, 1/10W Chip Resistor 0603 (1608 Metric) Automotive AEC-Q200 Thick Film"
 			(at 317.5 123.19 0)
 			(hide yes)
@@
 			)
 		)
-		(property "MPN" "RMCF0603FT100K"
+		(property "MPN" "RMCF0603FT10K0"
 			(at 317.5 123.19 0)
 			(hide yes)
@@
 			)
 		)
-		(property "DPN" "RMCF0603FT100KCT-ND"
+		(property "DPN" "RMCF0603FT10K0CT-ND"
 			(at 317.5 123.19 0)
 			(hide yes)
@@
 			)
 		)
-		(property "MFR" "Panasonic"
+		(property "MFR" "Stackpole Electronics"
 			(at 317.5 123.19 0)
 			(hide yes)
@@
 			)
 		)
-		(property "Value" "100n"
+		(property "Value" "0.1u"
 			(at 325.12 137.16 0)
 			(show_name no)
@@
 			)
 		)
-		(property "Datasheet" ""
+		(property "Datasheet" "https://search.kemet.com/download/specsheet/C0603C104K5RACAUTO"
 			(at 317.5 133.35 0)
 			(hide yes)
@@
 			)
 		)
-		(property "Description" "CAP CER 0.1UF 25V X7R 0603"
+		(property "Description" "0.1 µF ±10% 50V Ceramic Capacitor X7R 0603 (1608 Metric)"
 			(at 317.5 133.35 0)
 			(hide yes)
@@
 			)
 		)
-		(property "MPN" "CGA3E2X7R1E104K080AA"
+		(property "MPN" "C0603C104K5RACAUTO"
 			(at 317.5 133.35 0)
 			(hide yes)
@@
 			)
 		)
-		(property "DPN" "445-5667-1-ND"
+		(property "DPN" "399-6856-1-ND"
 			(at 317.5 133.35 0)
 			(hide yes)
@@
 			)
 		)
-		(property "MFR" "TDK Corporation"
+		(property "MFR" "KEMET"
 			(at 317.5 133.35 0)
 			(hide yes)
@@
 			)
 		)
-		(property "Value" "100n"
+		(property "Value" "0.1u"
 			(at 279.146 96.901 0)
 			(show_name no)
@@
 			)
 		)
-		(property "Datasheet" ""
+		(property "Datasheet" "https://search.kemet.com/download/specsheet/C0603C104K5RACAUTO"
 			(at 278.13 92.71 0)
 			(hide yes)
@@
 			)
 		)
-		(property "Description" "CAP CER 0.1UF 25V X7R 0603"
+		(property "Description" "0.1 µF ±10% 50V Ceramic Capacitor X7R 0603 (1608 Metric)"
 			(at 278.13 92.71 0)
 			(hide yes)
@@
 			)
 		)
-		(property "MPN" "CGA3E2X7R1E104K080AA"
+		(property "MPN" "C0603C104K5RACAUTO"
 			(at 278.13 92.71 0)
 			(hide yes)
@@
 			)
 		)
-		(property "DPN" "445-5667-1-ND"
+		(property "DPN" "399-6856-1-ND"
 			(at 278.13 92.71 0)
 			(hide yes)
@@
 			)
 		)
-		(property "MFR" "TDK Corporation"
+		(property "MFR" "KEMET"
 			(at 278.13 92.71 0)
 			(hide yes)
@@
 			)
 		)
-		(property "Datasheet" ""
+		(property "Datasheet" "https://www.seielect.com/catalog/SEI-RMCF_RMCP.pdf"
 			(at 181.61 88.9 0)
 			(hide yes)
@@
 			)
 		)
-		(property "Description" "Resistor, small US symbol"
+		(property "Description" "1 MOhms ±1% 0.1W, 1/10W Chip Resistor 0603 (1608 Metric) Automotive AEC-Q200 Thick Film"
 			(at 181.61 88.9 0)
 			(hide yes)
@@
 			)
 		)
-		(property "MPN" "ERJ-3EKF1004V"
+		(property "MPN" "RMCF0603FT1M00"
 			(at 181.61 88.9 0)
 			(hide yes)
@@
 			)
 		)
-		(property "DPN" "P1.00MHCT-ND"
+		(property "DPN" "RMCF0603FT1M00CT-ND"
 			(at 181.61 88.9 0)
 			(hide yes)
@@
 			)
 		)
-		(property "MFR" "Panasonic"
+		(property "MFR" "Stackpole Electronics"
 			(at 181.61 88.9 0)
 			(hide yes)
@@
 			)
 		)
-		(property "Datasheet" ""
+		(property "Datasheet" "https://datasheets.kyocera-avx.com/AutoMLCCKAM.pdf"
 			(at 163.83 111.76 0)
 			(hide yes)
@@
 			)
 		)
-		(property "MPN" "CGA3E2C0G1H120J080AA"
+		(property "MPN" "KAM15ACG2A120KT"
 			(at 163.83 111.76 0)
 			(hide yes)
@@
 			)
 		)
-		(property "DPN" "445-5629-1-ND"
+		(property "DPN" "478-KAM15ACG2A120KTTR-ND"
 			(at 163.83 111.76 90)
 			(hide yes)
@@
 			)
 		)
-		(property "MFR" "TDK Corporation"
+		(property "MFR" "KYOCERA AVX"
 			(at 163.83 111.76 90)
 			(hide yes)
@@
 			)
 		)
-		(property "Datasheet" ""
+		(property "Datasheet" "https://datasheets.kyocera-avx.com/AutoMLCCKAM.pdf"
 			(at 163.83 127 0)
 			(hide yes)
@@
 			)
 		)
-		(property "MPN" "CGA3E2C0G1H120J080AA"
+		(property "MPN" "KAM15ACG2A120KT"
 			(at 163.83 127 0)
 			(hide yes)
@@
 			)
 		)
-		(property "DPN" "445-5629-1-ND"
+		(property "DPN" "478-KAM15ACG2A120KTTR-ND"
 			(at 163.83 127 90)
 			(hide yes)
@@
 			)
 		)
-		(property "MFR" "TDK Corporation"
+		(property "MFR" "KYOCERA AVX"
 			(at 163.83 127 90)
 			(hide yes)
@@
 			)
 		)
-		(property "Datasheet" ""
+		(property "Datasheet" "https://datasheets.kyocera-avx.com/AutoMLCCKAM.pdf"
 			(at 156.21 81.28 0)
 			(hide yes)
@@
 			)
 		)
-		(property "MPN" "CGA3E2C0G1H120J080AA"
+		(property "MPN" "KAM15ACG2A120KT"
 			(at 156.21 81.28 0)
 			(hide yes)
@@
 			)
 		)
-		(property "DPN" "445-5629-1-ND"
+		(property "DPN" "478-KAM15ACG2A120KTTR-ND"
 			(at 156.21 81.28 90)
 			(hide yes)
@@
 			)
 		)
-		(property "MFR" "TDK Corporation"
+		(property "MFR" "KYOCERA AVX"
 			(at 156.21 81.28 90)
 			(hide yes)
@@
 			)
 		)
-		(property "Value" "100n"
+		(property "Value" "0.1u"
 			(at 154.686 187.071 0)
 			(show_name no)
@@
 			)
 		)
-		(property "Datasheet" ""
+		(property "Datasheet" "https://search.kemet.com/download/specsheet/C0603C104K5RACAUTO"
 			(at 153.67 182.88 0)
 			(hide yes)
@@
 			)
 		)
-		(property "Description" "CAP CER 0.1UF 25V X7R 0603"
+		(property "Description" "0.1 µF ±10% 50V Ceramic Capacitor X7R 0603 (1608 Metric)"
 			(at 153.67 182.88 0)
 			(hide yes)
@@
 			)
 		)
-		(property "MPN" "CGA3E2X7R1E104K080AA"
+		(property "MPN" "C0603C104K5RACAUTO"
 			(at 153.67 182.88 0)
 			(hide yes)
@@
 			)
 		)
-		(property "DPN" "445-5667-1-ND"
+		(property "DPN" "399-6856-1-ND"
 			(at 153.67 182.88 0)
 			(hide yes)
@@
 			)
 		)
-		(property "MFR" "TDK Corporation"
+		(property "MFR" "KEMET"
 			(at 153.67 182.88 0)
 			(hide yes)
@@
 			)
 		)
-		(property "Datasheet" ""
+		(property "Datasheet" "https://www.seielect.com/catalog/SEI-RMCF_RMCP.pdf"
 			(at 288.29 180.34 0)
 			(hide yes)
@@
 			)
 		)
-		(property "Description" "Resistor, small US symbol"
+		(property "Description" "0 Ohms Jumper Chip Resistor 0603 (1608 Metric) Automotive AEC-Q200 Thick Film"
 			(at 288.29 180.34 0)
 			(hide yes)
@@
 			)
 		)
-		(property "MPN" "ERJ-3GEY0R00V"
+		(property "MPN" "RMCF0603ZT0R00"
 			(at 288.29 180.34 0)
 			(hide yes)
@@
 			)
 		)
-		(property "DPN" "P0.0GCT-ND"
+		(property "DPN" "RMCF0603ZT0R00CT-ND"
 			(at 288.29 180.34 0)
 			(hide yes)
@@
 			)
 		)
-		(property "MFR" "Panasonic"
+		(property "MFR" "Stackpole Electronics"
 			(at 288.29 180.34 0)
 			(hide yes)
@@
 			)
 		)
-		(property "Datasheet" ""
+		(property "Datasheet" "https://datasheets.kyocera-avx.com/AutoMLCCKAM.pdf"
 			(at 156.21 96.52 0)
 			(hide yes)
@@
 			)
 		)
-		(property "MPN" "CGA3E2C0G1H120J080AA"
+		(property "MPN" "KAM15ACG2A120KT"
 			(at 156.21 96.52 0)
 			(hide yes)
@@
 			)
 		)
-		(property "DPN" "445-5629-1-ND"
+		(property "DPN" "478-KAM15ACG2A120KTTR-ND"
 			(at 156.21 96.52 90)
 			(hide yes)
@@
 			)
 		)
-		(property "MFR" "TDK Corporation"
+		(property "MFR" "KYOCERA AVX"
 			(at 156.21 96.52 90)
 			(hide yes)
